File: Electrical/Pico Shield/pico_shield_ver1/pico_shield_ver1.kicad_sch (KiCad schematic)
At the start: 5 parts, among them U1 pico_shield, U2 ULN2003A, U3 ULN2003A

Commit message: reorg
Parts:
- removed C1: 10n, symbol Device:C
- removed U1: pico_shield, symbol pi_pico_shield:pico_shield
- added C?: 10n, symbol Device:C
- added U?: pico_shield, symbol pi_pico_shield:pico_shield
Connections:
- net +5V: now also C?.2
- net GND: now also C?.1
Other:
- moved on the sheet: C2, U2, U3

Commit message: I need more commits than Gavin
Parts:
- added J? (x2): Step_connector, Connector_JST:JST_XH_B5B-XH-A_1x05_P2.50mm_Vertical, symbol dk_Rectangular-Connectors-Headers-Male-Pins:B5B-XH-A_LF__SN_
Connections:
- net +5V: now also J?.1, J?.1
- net GND: now also U?.13 (GND), U?.18 (GND), U?.23 (GND), U?.3 (GND), U?.33 (GND), U?.38 (GND), U?.8 (GND); no longer U2.10 (O7), U2.11 (O6), U2.12 (O5), U2.5 (I5), U2.6 (I6), U2.7 (I7), U3.10 (O7), U3.11 (O6), U3.12 (O5), U3.5 (I5), U3.6 (I6), U3.7 (I7)
- net Motor - Blue: now also U?.27 (GP21)
- net Motor - Orange: now also U?.19 (GP14), U?.24 (GP18)
- net Motor - Pink: now also U?.21 (GP16), U?.22 (GP17), U?.26 (GP20)
- net Motor - Yellow: now also U?.20 (GP15), U?.25 (GP19)
- net at U2.1 (I1): now also J?.2
- net at U2.2 (I2): now also J?.3
- net at U2.3 (I3): now also J?.4
- net at U2.4 (I4): now also J?.5
- net at U3.1 (I1): now also J?.2
- net at U3.2 (I2): now also J?.3
- net at U3.3 (I3): now also J?.4
- net at U3.4 (I4): now also J?.5
- no-connect marks 0 -> 12

Commit message: Almost Complete rough draft
Doesn't have my custom footprint for components not on PCB, but on BOM such as connectors
Parts:
- added EXT? (x8): Photodiode male connector (8), 0_custom:EXT_no_footprint, symbol 0_custom:{lt}name{gt}
- added EXT?: Photodiodes (8), 0_custom:EXT_no_footprint, symbol 0_custom:{lt}name{gt}
- added EXT?: Power Male Connector, 0_custom:EXT_no_footprint, symbol 0_custom:{lt}name{gt}
- added EXT?: PWR Banana Plugs, 0_custom:EXT_no_footprint, symbol 0_custom:{lt}name{gt}
- added J?: 644752-2, Miles Added:644752-2_TYC, symbol dk_Rectangular-Connectors-Headers-Male-Pins:B2B-PH-K-S_LF__SN_
- added J? (x8): B2B-PH-K-S_LF__SN_, digikey-footprints:PinHeader_1x2_P2mm_Drill1mm, symbol dk_Rectangular-Connectors-Headers-Male-Pins:B2B-PH-K-S_LF__SN_
- added R? (x8): 1M, symbol Device:R_US
- added R?: 180k, symbol Device:R_US
- added R?: 10k, symbol Device:R_US
- added U?: CD4051B, symbol Analog_Switch:CD4051B
- added U?: LM358, symbol Amplifier_Operational:LM358
Connections:
- net +5V: now also U?.39 (VSYS), J?.1, R?.1, R?.1, R?.1, R?.1, U?.16 (VDD)
- net GND: now also J?.2, J?.2, J?.2, J?.2, J?.2, J?.2, J?.2, J?.2, J?.2, R?.1, U?.6 (INH), U?.7 (VEE), U?.8 (VSS)
- net MCU GPIO (S0): now reaches U?.15 (GP11)
- net MCU GPIO (S0): now also U?.11 (A)
- net MCU GPIO (S1): now reaches U?.16 (GP12)
- net MCU GPIO (S1): now also U?.10 (B)
- net MCU GPIO (S2): now reaches U?.17 (GP13)
- net MCU GPIO (S2): now also U?.9 (C)
- net MCU ADC: now reaches U?.34 (GP28)
- net MCU ADC: now also R?.2, U?.1
- new net: R?.1, R?.1, R?.1, R?.1
- new net: U?.3 (+), U?.3 (X)
- new net: R?.1, R?.2, U?.2 (-)
- new net PhDio_0: J?.1, R?.2, U?.13 (X0)
- new net PhDio_1: J?.1, R?.2, U?.14 (X1)
- new net PhDio_2: J?.1, R?.2, U?.15 (X2)
- new net PhDio_3: R?.2, U?.12 (X3)
- new net PhDio_4: J?.1, R?.2, U?.1 (X4)
- new net PhDio_5: J?.1, R?.2, U?.5 (X5)
- new net PhDio_6: J?.1, R?.2, U?.2 (X6)
- new net PhDio_7: R?.2, U?.4 (X7)
Other:
- note added: "Positioning Photodiodes for CubeSat Corners"
- note added: "RPi Shield"
- note added: "Step Motor Drivers"
- note added: "todo: - power input - ptc over current protection? - no footprint components for BOM - photodiodes - custom shield footprint"
- moved on the sheet: C2, C?, J?, U2, U3, U?

Commit message: progress
Parts:
- removed C?: 10n, symbol Device:C
- removed R? (x7): 1M, symbol Device:R_US
- removed U2: ULN2003A, symbol Transistor_Array:ULN2003A
- added C1: 2.2uF Cer., Capacitor_SMD:C_0805_2012Metric, symbol Device:C
- added C3: 4.7uF Cer., Capacitor_SMD:C_0805_2012Metric, symbol Device:C
- added C4: 10n, Capacitor_SMD:C_0805_2012Metric, symbol Device:C
- added EXT3: 2nd set of pico headers, 0_custom:EXT_no_footprint, symbol 0_custom:{lt}name{gt}
- added EXT5: Pico Headers, 0_custom:EXT_no_footprint, symbol 0_custom:{lt}name{gt}
- added EXT7: NiCr Wire Connector, 0_custom:EXT_no_footprint, symbol 0_custom:{lt}name{gt}
- added J1: 644752-2, Miles Added:644752-2_TYC, symbol dk_Rectangular-Connectors-Headers-Male-Pins:B2B-PH-K-S_LF__SN_
- added R1: 15k, Resistor_SMD:R_0805_2012Metric_Pad1.20x1.40mm_HandSolder, symbol Device:R_US
- added R10, R11, R12, R13, R5, R6, R7: 1M, Resistor_SMD:R_0805_2012Metric_Pad1.20x1.40mm_HandSolder, symbol Device:R_US
- added R2: 7k8, Resistor_SMD:R_0805_2012Metric_Pad1.20x1.40mm_HandSolder, symbol Device:R_US
- added R3: 47k, Resistor_SMD:R_0805_2012Metric_Pad1.20x1.40mm_HandSolder, symbol Device:R_US
- added U1: XC6230A001QR-G, Miles Added:SOIC127P600X175-9N, symbol XC6230A001QR-G:XC6230A001QR-G
- added U2: Si1442DH, Package_TO_SOT_SMD:SOT-363_SC-70-6, symbol 0_custom:Si1442DH
- added U4: ULN2003A, Miles Added:ULN2003ADR2G_OSI, symbol Transistor_Array:ULN2003A
- C2: footprint (none) -> Capacitor_SMD:C_0805_2012Metric; MPN (none) -> 0805YC103MAT2A
- R4: renamed from R?; footprint (none) -> Resistor_SMD:R_0805_2012Metric_Pad1.20x1.40mm_HandSolder; MPN (none) -> RT0805BRD071ML
- R8: renamed from R?; footprint (none) -> Resistor_SMD:R_0805_2012Metric_Pad1.20x1.40mm_HandSolder; MPN (none) -> RC0805FR-07182KL
- R9: renamed from R?; footprint (none) -> Resistor_SMD:R_0805_2012Metric_Pad1.20x1.40mm_HandSolder; MPN (none) -> RMCF0805FT10K0
- U3: footprint (none) -> Miles Added:ULN2003ADR2G_OSI; MPN (none) -> ULN2003ADR2G
- U5: renamed from U?; footprint (none) -> 0_custom:PICO_SHIELD; MPN (none) -> PRT-16279
- U6: renamed from U?; footprint (none) -> Miles Added:M08A-L; MPN (none) -> LM358MX
- U7: renamed from U?; footprint (none) -> Miles Added:PW0016A_L; MPN (none) -> CD4051BQPWRG4Q1
- gave numbers to parts that had none: 22
Connections:
- net +5V: now also C1.1, C4.2, R5.1, R6.1, R7.1, U1.8 (VIN), U4.9 (COM)
- net GND: now also C1.2, C3.2, C4.1, R2.1, R3.1, U1.6 (VSS), U2.4 (S), U4.8 (GND)
- net Motor - Blue: now also U4.13 (O4)
- net Motor - Orange: now also U4.16 (O1)
- net Motor - Pink: now also U4.14 (O3)
- net Motor - Yellow: now also U4.15 (O2)
- net PhDio_1: now also R5.2
- net PhDio_2: now also R6.2
- net PhDio_3: now also J12.1, R7.2
- net PhDio_4: now also R13.2
- net PhDio_5: now also R12.2
- net PhDio_6: now also R11.2
- net PhDio_7: now also J11.1, R10.2
- net at J4.2: now also U4.1 (I1)
- net at J4.3: now also U4.2 (I2)
- net at J4.4: now also U4.3 (I3)
- net at J4.5: now also U4.4 (I4)
- net LDO_EN: now reaches U5.11 (GP8)
- net LDO_EN: now also U1.5 (CE)
- net Burn_sig: now reaches U5.12 (GP9)
- net Burn_sig: now also U2.3 (G)
- new net: R1.1, R3.2, U1.4 (VOFB)
- new net: R10.1, R11.1, R12.1, R13.1
- new net: U1.2 (NC), U1.7 (NC)
- new net: R2.2, U1.3 (ILIM)
- new net NiCr_HS: C3.1, J1.1, R1.2, U1.1 (VOUT)
- new net NiCr_LS: J1.2, U2.1 (D), U2.2 (D), U2.5 (D), U2.6 (D)
- no-connect marks 12 -> 30
Other:
- note added: "NiChrome Wire Burner"
- note added: "Other Components"
- note added: "Power Supply Input"
- note added: "todo: - power input - overcurrent and overvoltage protection - no footprint components for BOM - photodiodes - custom shield footprint - test points - gnd pin to clip to - add connection points for photodiode breakout boards"
- note removed: "todo: - power input - ptc over current protection? - no footprint components for BOM - photodiodes - custom shield footprint"
- company: (none) -> Cal Poly, SLO
- title: (none) -> CubeSat Pi Hat
- moved on the sheet: C2, EXT1, EXT10, EXT11, EXT12, EXT13, EXT14, EXT2, EXT4, EXT6, EXT8, EXT9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

Commit message: mo' progress
Parts:
- added J3, J6: B5B-XH-A_LF__SN_, digikey-footprints:PinHeader_1x5_P2.5mm_Drill1.1mm, symbol dk_Rectangular-Connectors-Headers-Male-Pins:B5B-XH-A_LF__SN_
- added TP1, TP2: TestPoint, symbol Connector:TestPoint
- J1: footprint Miles Added:644752-2_TYC -> digikey-footprints:PinHeader_1x2_P2mm_Drill1mm; DK_Datasheet_Link (none) -> http://www.jst-mfg.com/product/pdf/eng/ePH.pdf; DK_Detail_Page (none) -> /product-detail/en/jst-sales-america-inc/B2B-PH-K-S(LF)(SN)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; Digi-Key_PN (none) -> 455-1704-ND; MPN 644752-2 -> B2B-PH-K-S(LF)(SN); Manufacturer (none) -> JST Sales America Inc.
- J2: footprint Connector_JST:JST_XH_B5B-XH-A_1x05_P2.50mm_Vertical -> digikey-footprints:PinHeader_1x5_P2.5mm_Drill1.1mm; Category (none) -> Connectors, Interconnects; DK_Datasheet_Link (none) -> http://www.jst-mfg.com/product/pdf/eng/eXH.pdf; DK_Detail_Page (none) -> /product-detail/en/jst-sales-america-inc/B5B-XH-A(LF)(SN)/4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; Digi-Key_PN (none) -> 455-2270-ND; Family (none) -> Rectangular Connectors - Headers, Male Pins; Manufacturer (none) -> JST Sales America Inc.; Status (none) -> Active
- J4: renamed from J3; footprint Miles Added:644752-2_TYC -> digikey-footprints:PinHeader_1x2_P2mm_Drill1mm; DK_Datasheet_Link (none) -> http://www.jst-mfg.com/product/pdf/eng/ePH.pdf; DK_Detail_Page (none) -> /product-detail/en/jst-sales-america-inc/B2B-PH-K-S(LF)(SN)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; Digi-Key_PN (none) -> 455-1704-ND; MPN 644752-2 -> B2B-PH-K-S(LF)(SN); Manufacturer (none) -> JST Sales America Inc.
- J5: renamed from J4; footprint Connector_JST:JST_XH_B5B-XH-A_1x05_P2.50mm_Vertical -> digikey-footprints:PinHeader_1x5_P2.5mm_Drill1.1mm; Category (none) -> Connectors, Interconnects; DK_Datasheet_Link (none) -> http://www.jst-mfg.com/product/pdf/eng/eXH.pdf; DK_Detail_Page (none) -> /product-detail/en/jst-sales-america-inc/B5B-XH-A(LF)(SN)/4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; Digi-Key_PN (none) -> 455-2270-ND; Family (none) -> Rectangular Connectors - Headers, Male Pins; Manufacturer (none) -> JST Sales America Inc.; Status (none) -> Active
- U1: footprint Miles Added:SOIC127P600X175-9N -> SOIC127P600X175-9N; SNAPEDA_PN (none) -> XC6230H001QR-G
- U5: footprint 0_custom:PICO_SHIELD -> (none); MPN PRT-16279 -> (none)
- renumbered C2 to C1, C1 to C2, J5 to J10, J9 to J11, J10 to J12, J7 to J13, J11 to J14, J6 to J7, J12 to J8, J8 to J9, U7 to U6, U6 to U7
Connections:
- net +5V: now also TP2.1
- net Burn_sig: now also U5.19 (GP14); no longer U5.12 (GP9)
- net GND: no longer U5.33 (GND)
- net LDO_EN: now also U5.20 (GP15); no longer U5.11 (GP8)
- net NiCr_HS: now also TP1.1
- net MTR1 - Yellow: now reaches U5.10 (GP7)
- net MTR1 - Yellow: now also U3.15 (O2)
- net MTR2 - Orange: now reaches U5.14 (GP10)
- net MTR2 - Orange: now also U4.16 (O1)
- net PDBO_ADC_1: now reaches U5.31 (GP26)
- net PDBO_ADC_1: now also J3.1
- net PDBO_ADC_2: now reaches U5.32 (GP27)
- net PDBO_ADC_2: now also J6.1
- net +3.3VADC: now reaches U5.35 (ADC_VREF)
- net +3.3VADC: now also J3.4, J6.4
- net MUX (S0): now reaches U5.5 (GP3)
- net MUX (S0): now also U6.11 (A)
- net MUX (S1): now reaches U5.6 (GP4)
- net MUX (S1): now also U6.10 (B)
- net MUX (S2): now reaches U5.7 (GP5)
- net MUX (S2): now also U6.9 (C)
- net MTR1 - Orange: now reaches U5.9 (GP6)
- net MTR1 - Orange: now also U3.16 (O1)
- net at U1.2 (NC): no longer U1.7 (NC)
- net MCU GPIO (S0) renamed MTR2 - Yellow
- net MTR2 - Yellow: now also U4.15 (O2); no longer U6.11 (A)
- net MCU GPIO (S1) renamed MTR2 - Pink
- net MTR2 - Pink: now also U4.14 (O3); no longer U6.10 (B)
- net MCU GPIO (S2) renamed MTR2 - Blue
- net MTR2 - Blue: now also U4.13 (O4); no longer U6.9 (C)
- removed net Motor - Blue: U3.13 (O4), U4.13 (O4), U5.27 (GP21)
- removed net Motor - Orange: U3.16 (O1), U4.16 (O1), U5.19 (GP14), U5.24 (GP18)
- removed net Motor - Pink: U3.14 (O3), U4.14 (O3), U5.21 (GP16), U5.22 (GP17), U5.26 (GP20)
- removed net Motor - Yellow: U3.15 (O2), U4.15 (O2), U5.20 (GP15), U5.25 (GP19)
- new net GNDA: J3.5, J6.5, U5.33 (ADC_GND)
- new net MTR1 - Blue: U3.13 (O4), U5.12 (GP9)
- new net MTR1 - Pink: U3.14 (O3), U5.11 (GP8)
- new net PDBO_MUX_1_1: J3.2, U5.25 (GP19)
- new net PDBO_MUX_1_2: J3.3, U5.24 (GP18)
- new net PDBO_MUX_2_1: J6.2, U5.27 (GP21)
- new net PDBO_MUX_2_2: J6.3, U5.26 (GP20)
- no-connect marks 30 -> 23
Other:
- note added: "Based on ______ Stepper motor drivers"
- note added: "Headers to external photodiodes"
- note added: "Photodiode Breakout Connectors"
- note added: "TODO: - Powering the PICO"
- note removed: "todo: - power input - overcurrent and overvoltage protection - no footprint components for BOM - photodiodes - custom shield footprint - test points - gnd pin to clip to - add connection points for photodiode breakout boards"
- moved on the sheet: C1, C2, C3, EXT1, EXT10, EXT11, EXT12, EXT13, EXT14, EXT2, EXT3, EXT4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

Commit message: Draft 1 Schematic, Awaiting Review
Connections:
- net +5V: no longer R4.1, R5.1, R6.1, R7.1, U6.16 (VDD)
- net +3.3V: now reaches U5.36 (3V3)
- net +3.3V: now also R4.1, R5.1, R6.1, R7.1, U6.16 (VDD)
- no-connect marks 23 -> 22
Other:
- note added: "Need diode on VSYS?"
- note removed: "Based on ______ Stepper motor drivers"
Changed lines of the file:
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@@
   (junction (at 108.585 190.5) (diameter 0) (color 0 0 0 0)
   )
-  (junction (at 71.12 142.24) (diameter 0) (color 0 0 0 0)
-  )
   (junction (at 46.99 175.26) (diameter 0) (color 0 0 0 0)
   )
@@
   (no_connect (at 44.45 106.68))
   (no_connect (at 246.38 131.445))
-  (no_connect (at 246.38 113.665))
   (no_connect (at 64.77 106.68))
   (no_connect (at 64.77 101.6))
@@
     (stroke (width 0) (type default) (color 0 0 0 0))
   )
-  (wire (pts (xy 71.12 142.24) (xy 71.12 143.51))
+  (wire (pts (xy 71.12 139.7) (xy 71.12 143.51))
     (stroke (width 0) (type default) (color 0 0 0 0))
   )
@@
     (stroke (width 0) (type default) (color 0 0 0 0))
   )
+  (wire (pts (xy 246.38 113.665) (xy 248.92 113.665))
+    (stroke (width 0) (type default) (color 0 0 0 0))
+  )
   (wire (pts (xy 68.58 43.18) (xy 68.58 46.99))
     (stroke (width 0) (type default) (color 0 0 0 0))
@@
     (stroke (width 0) (type default) (color 0 0 0 0))
   )
-  (wire (pts (xy 71.12 139.7) (xy 71.12 142.24))
-    (stroke (width 0) (type default) (color 0 0 0 0))
-  )
   (wire (pts (xy 246.38 133.985) (xy 248.92 133.985))
     (stroke (width 0) (type default) (color 0 0 0 0))
@@
     (stroke (width 0) (type default) (color 0 0 0 0))
   )
-  (wire (pts (xy 71.12 138.43) (xy 71.12 139.7))
+  (wire (pts (xy 71.12 136.525) (xy 71.12 139.7))
     (stroke (width 0) (type default) (color 0 0 0 0))
   )
@@
     (effects (font (size 2 2)) (justify left bottom))
   )
-  (text "Based on ______ Stepper motor drivers\n" (at 20.955 38.735 270)
-    (effects (font (size 1.27 1.27)) (justify right bottom))
-  )
   (text "NiChrome Wire Burner\n" (at 179.07 26.67 0)
     (effects (font (size 2 2)) (justify left bottom))
@@
     (effects (font (size 1.27 1.27)) (justify left bottom))
   )
+  (text "Need diode on VSYS?" (at 271.78 102.235 180)
+    (effects (font (size 1.27 1.27)) (justify right bottom))
+  )
   (text "Step Motor Drivers" (at 53.975 33.02 0)
     (effects (font (size 2 2)) (justify left bottom))
@@
     (pin "2")
   )
+  (symbol (lib_id "power:+3.3V") (at 71.12 136.525 90) (unit 1)
+    (in_bom yes) (on_board yes) (fields_autoplaced)
+    (property "Reference" "#PWR?" (id 0) (at 74.93 136.525 0)
+      (effects (font (size 1.27 1.27)) hide)
+    )
+    (property "Value" "+3.3V" (id 1) (at 72.39 136.5249 90)
+      (effects (font (size 1.27 1.27)) (justify right))
+    )
+    (property "Footprint" "" (id 2) (at 71.12 136.525 0)
+      (effects (font (size 1.27 1.27)) hide)
+    )
+    (property "Datasheet" "" (id 3) (at 71.12 136.525 0)
+      (effects (font (size 1.27 1.27)) hide)
+    )
+    (pin "1")
+  )
   (symbol (lib_id "power:+5V") (at 257.81 106.045 270) (unit 1)
     (in_bom yes) (on_board yes)
@@
     (pin "1")
   )
-  (symbol (lib_id "power:+5V") (at 71.12 138.43 0) (unit 1)
-    (in_bom yes) (on_board yes)
-    (property "Reference" "#PWR033" (id 0) (at 71.12 142.24 0)
-      (effects (font (size 1.27 1.27)) hide)
-    )
-    (property "Value" "+5V" (id 1) (at 71.12 134.62 0))
-    (property "Footprint" "" (id 2) (at 71.12 138.43 0)
-      (effects (font (size 1.27 1.27)) hide)
-    )
-    (property "Datasheet" "" (id 3) (at 71.12 138.43 0)
-      (effects (font (size 1.27 1.27)) hide)
-    )
-    (pin "1")
-  )
   (symbol (lib_id "power:+5V") (at 68.58 85.09 0) (mirror y) (unit 1)
     (in_bom yes) (on_board yes) (fields_autoplaced)
@@
   )
   (symbol (lib_id "pi_pico_shield:pico_shield") (at 215.9 106.045 0) (unit 1)
-    (in_bom yes) (on_board yes) (fields_autoplaced)
-    (property "Reference" "U5" (id 0) (at 226.695 93.98 0))
-    (property "Value" "pico_shield" (id 1) (at 226.695 96.52 0))
+    (in_bom yes) (on_board yes)
+    (property "Reference" "U5" (id 0) (at 226.695 118.745 0))
+    (property "Value" "pico_shield" (id 1) (at 226.695 116.205 0))
     (property "Footprint" "" (id 2) (at 215.9 106.045 0)
       (effects (font (size 1.27 1.27)) hide)
@@
     (pin "2")
   )
-  (symbol (lib_id "power:PWR_FLAG") (at 71.12 142.24 90) (unit 1)
-    (in_bom yes) (on_board yes) (fields_autoplaced)
-    (property "Reference" "#FLG01" (id 0) (at 69.215 142.24 0)
-      (effects (font (size 1.27 1.27)) hide)
-    )
-    (property "Value" "PWR_FLAG" (id 1) (at 67.31 142.2399 90)
-      (effects (font (size 1.27 1.27)) (justify left))
-    )
-    (property "Footprint" "" (id 2) (at 71.12 142.24 0)
-      (effects (font (size 1.27 1.27)) hide)
-    )
-    (property "Datasheet" "~" (id 3) (at 71.12 142.24 0)
-      (effects (font (size 1.27 1.27)) hide)
-    )
-    (pin "1")
-  )
   (symbol (lib_id "Device:R_US") (at 46.99 181.61 0) (mirror x) (unit 1)
     (in_bom yes) (on_board yes)
@@
     (pin "2")
   )
+  (symbol (lib_id "power:+3.3V") (at 248.92 113.665 270) (unit 1)
+    (in_bom yes) (on_board yes) (fields_autoplaced)
+    (property "Reference" "#PWR?" (id 0) (at 245.11 113.665 0)
+      (effects (font (size 1.27 1.27)) hide)
+    )
+    (property "Value" "+3.3V" (id 1) (at 252.73 113.6649 90)
+      (effects (font (size 1.27 1.27)) (justify left))
+    )
+    (property "Footprint" "" (id 2) (at 248.92 113.665 0)
+      (effects (font (size 1.27 1.27)) hide)
+    )
+    (property "Datasheet" "" (id 3) (at 248.92 113.665 0)
+      (effects (font (size 1.27 1.27)) hide)
+    )
+    (pin "1")
+  )
   (symbol (lib_id "dk_Rectangular-Connectors-Headers-Male-Pins:B2B-PH-K-S_LF__SN_") (at 113.03 128.905 90) (mirror x) (unit 1)
     (in_bom yes) (on_board yes) (fields_autoplaced)
@@
   )
   (symbol_instances
-    (path "/b6b931a3-6cd6-40bc-9365-c77a25f59059"
-      (reference "#FLG01") (unit 1) (value "PWR_FLAG") (footprint "")
-    )
     (path "/501f0b31-86ce-46d3-9de6-93e0fe1365dd"
       (reference "#PWR01") (unit 1) (value "+5V") (footprint "")
@@
       (reference "#PWR032") (unit 1) (value "GND") (footprint "")
     )
-    (path "/9d75283d-ddfe-416c-9ed4-a77efabfe370"
-      (reference "#PWR033") (unit 1) (value "+5V") (footprint "")
-    )
     (path "/c168e9cc-09b4-49db-b745-acadf29006f7"
       (reference "#PWR034") (unit 1) (value "GND") (footprint "")
@@
       (reference "#PWR038") (unit 1) (value "GND") (footprint "")
     )
+    (path "/2bef4b8b-ea01-4399-965f-be6881cd9329"
+      (reference "#PWR?") (unit 1) (value "+3.3V") (footprint "")
+    )
+    (path "/b9577cd0-65dc-44f9-a34f-7ce9f80f5cc3"
+      (reference "#PWR?") (unit 1) (value "+3.3V") (footprint "")
+    )
     (path "/5e66c672-3d40-4610-b736-35555b442c18"
