File: Electrical/SADA_Board/SADA_Board/SADA_Board.kicad_pcb (KiCad board)
At the start: 4 copper layers, 85 x 50 mm, 125 parts, among them IC1 TPS25940LRVCR, IC2 LP5912Q3.3DRVRQ1, J1 Headers, J10 171973-0004, J11 105431-1202, J12 105431-1202, J2 Aux. Photodiode Board 1, J3 Aux. Photodiode Board 2, J4 Systems Board Connector, J5 Conn_01x05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

Commit message: ESD changes
Parts:
- removed EXT11: NiCr Wire Connector, 0_custom:EXT_no_footprint
- removed the EXT4 at (132.6, 39.3)
- removed J12: 105431-1202, Miles Added:1054311202
- removed U10, U9: Si1442DH, Package_TO_SOT_SMD:SOT-363_SC-70-6
- added C33: 100nF, Capacitor_SMD:C_0402_1005Metric, F.Cu at (152.9, 57.9)
- added D1: TVS, Diode_SMD:D_0402_1005Metric, F.Cu at (154.2, 121.4)
- added D10: TVS, Diode_SMD:D_0402_1005Metric, F.Cu at (182.2, -104.4)
- added D11: TVS, Diode_SMD:D_0402_1005Metric, F.Cu at (182.2, -102.4)
- added D14: TVS, Diode_SMD:D_0402_1005Metric, F.Cu at (180.4, -115.8)
- added D15: TVS, Diode_SMD:D_0402_1005Metric, F.Cu at (186.6, -113.8)
- added D16: TVS, Diode_SMD:D_0402_1005Metric, F.Cu at (183.5, -113.8)
- added D17: TVS, Diode_SMD:D_0402_1005Metric, F.Cu at (183.5, -109.9)
- added D18: TVS, Diode_SMD:D_0402_1005Metric, F.Cu at (177.2, -115.8)
- added D19: TVS, Diode_SMD:D_0402_1005Metric, F.Cu at (183.5, -115.8)
- added D2: TVS, Diode_SMD:D_0402_1005Metric, F.Cu at (146.4, 53.5)
- added D20: TVS, Diode_SMD:D_0402_1005Metric, F.Cu at (177.2, -109.9)
- added D21: TVS, Diode_SMD:D_0402_1005Metric, F.Cu at (180.4, -113.8)
- added D22: TVS, Diode_SMD:D_0402_1005Metric, F.Cu at (177.2, -113.8)
- added D23: TVS, Diode_SMD:D_0402_1005Metric, F.Cu at (186.6, -115.8)
- added D24: TVS, Diode_SMD:D_0402_1005Metric, F.Cu at (177.2, -111.9)
- added D25: TVS, Diode_SMD:D_0402_1005Metric, F.Cu at (180.4, -111.9)
- added D26: TVS, Diode_SMD:D_0402_1005Metric, F.Cu at (183.5, -111.9)
- added D27: TVS, Diode_SMD:D_0402_1005Metric, F.Cu at (180.4, -109.9)
- added D28: LG_R971-KN-1, digikey-footprints:0805, F.Cu at (122.9, 63.7)
- added D3: TVS, Diode_SMD:D_0402_1005Metric, F.Cu at (122.2, 66.6)
- added D4: TVS, Diode_SMD:D_0402_1005Metric, F.Cu at (128.4, 66.6)
- added D5: TVS, Diode_SMD:D_0402_1005Metric, F.Cu at (143.2, 53.5)
- added D6: TVS, Diode_SMD:D_0402_1005Metric, F.Cu at (125.3, 66.1)
- added D7: TVS, Diode_SMD:D_0402_1005Metric, F.Cu at (131.6, 66.6)
- added D8: TVS, Diode_SMD:D_0402_1005Metric, F.Cu at (195.2, -115.8)
- added H1: MountingHole_Pad, MountingHole:MountingHole_2.5mm_Pad, F.Cu at (4.00, -79.0)
- added H2: MountingHole_Pad, MountingHole:MountingHole_2.5mm_Pad, F.Cu at (4.00, -4.00)
- added H3: MountingHole_Pad, MountingHole:MountingHole_2.5mm_Pad, F.Cu at (79.0, -4.00)
- added H4: MountingHole_Pad, MountingHole:MountingHole_2.5mm_Pad, F.Cu at (79.0, -79.0)
- added JP1: Jumper_3_Open, Connector_PinHeader_2.54mm:PinHeader_1x03_P2.54mm_Vertical_SMD_Pin1Right, F.Cu at (124.4, 57.4)
- added Q3: IRLML6244TRPBF, Miles Added:SOT95P237X112-3N, F.Cu at (178.0, -103.1)
- added R31: 4.7k, Resistor_SMD:R_0402_1005Metric, F.Cu at (126.8, 63.2)
- added U11: USBLC6-2SC6, Package_TO_SOT_SMD:SOT-23-6, F.Cu at (154.0, 54.7)
- TP1, TP10, TP11, TP12, TP13, TP14, TP15, TP16, TP17, TP18, TP19, TP2, TP20, TP21, TP22, TP5, TP6, TP7, TP8, TP9: footprint TestPoint:TestPoint_Pad_D1.5mm -> TestPoint:TestPoint_Pad_D1.0mm
- TP3: renamed from TP4; footprint TestPoint:TestPoint_Pad_D1.5mm -> TestPoint:TestPoint_Pad_D1.0mm
- TP4: renamed from TP3; footprint TestPoint:TestPoint_Pad_D1.5mm -> TestPoint:TestPoint_Pad_D1.0mm
- moved J1 183.1 mm to (12.6, -80.5)
- moved J9 174.6 mm to (6.35, -67.3), turned to 90 degrees
- moved U1 172.0 mm to (41.4, -38.6)
- moved TP14 170.9 mm to (12.2, -71.4)
- moved TP16 168.5 mm to (12.2, -68.6)
- moved TP15 166.3 mm to (19.6, -75.2), turned to -90 degrees
- moved TP18 166.1 mm to (12.2, -65.5)
- moved TP19 163.6 mm to (12.2, -62.5)
- moved TP13 161.0 mm to (23.2, -73.5), turned to -90 degrees
- moved TP20 160.9 mm to (18.4, -68.1), turned to -90 degrees
- moved R16 159.1 mm to (16.6, -63.6), turned to -90 degrees
- moved U6 157.9 mm to (22.3, -69.3), turned to -90 degrees
- moved R14 156.6 mm to (19.6, -64.7), turned to 180 degrees
- moved R17 156.2 mm to (16.8, -71.4), turned to 180 degrees
- moved TP17 155.6 mm to (20.1, -72.2), turned to -90 degrees
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- renumbered D2 to D9, J5 to J4, J4 to J5
Connections:
- C12 pad 2: VBUS -> Net-(C12-Pad2)
- J8 pad 2: /USB_OTG_FS_DM -> /USB and MCU LDO/USB_CONN_DM
- J8 pad 3: /USB_OTG_FS_DP -> /USB and MCU LDO/USB_CONN_DP
- Q1 pad 2: VBUS -> Net-(C12-Pad2)
- TP3 pad 1: /SYS_SDA -> /SYS_SCL
- TP4 pad 1: /SYS_SCL -> /SYS_SDA
- TP7 pad 1: VBUS -> Net-(C12-Pad2)
- U4 pad 1: VBUS -> Net-(C12-Pad2)
Other:
- board size 85 x 50 mm -> 83 x 83 mm

Commit message: layout prog
Parts:
- removed D4, D5: TVS, Diode_SMD:D_0402_1005Metric
- J4: footprint Connector_PinSocket_2.00mm:PinSocket_1x05_P2.00mm_Vertical -> Connector_PinHeader_2.00mm:PinHeader_1x05_P2.00mm_Vertical_SMD_Pin1Left
- JP1: footprint Connector_PinHeader_2.54mm:PinHeader_1x03_P2.54mm_Vertical_SMD_Pin1Right -> Connector_PinHeader_2.00mm:PinHeader_1x03_P2.00mm_Vertical_SMD_Pin1Left
- moved D8 250.8 mm to (231.1, 132.3)
- moved D28 176.9 mm to (-35.1, -16.0)
- moved D3 176.9 mm to (-35.8, -13.1)
- moved D6 176.9 mm to (-32.7, -13.6)
- moved D7 176.9 mm to (-26.4, -13.1)
- moved JP1 176.9 mm to (-33.5, -22.4)
- moved R31 176.9 mm to (-31.2, -16.5)
- moved D14 175.5 mm to (13.2, -62.5), turned to -90 degrees
- moved D15 173.5 mm to (18.5, -70.8), turned to 90 degrees
- moved D19 170.7 mm to (21.1, -63.2), turned to -90 degrees
- moved D16 169.0 mm to (20.1, -70.8), turned to 90 degrees
- moved D17 165.0 mm to (23.4, -69.8)
- moved D18 161.8 mm to (23.4, -65.8)
- moved D20 158.3 mm to (26.2, -62.5)
- moved D10 145.7 mm to (195.1, 40.7)
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Connections:
- net /PA4 renamed /DAC_OUT1
- net /PA5 renamed /DAC_OUT2
- D18 pad 1: unconnected-(D18-Pad1) -> /MTR1_FAULT
Routing:
- net /Steppers /V_REF2: track 3.60 -> 0.00 mm

Commit message: layout prog
Parts:
- added C34: 22 uF, Capacitor_SMD:C_1210_3225Metric, F.Cu at (27.9, -80.3)
- added C35: 100nF, Capacitor_SMD:C_0402_1005Metric, F.Cu at (21.3, -81.3)
- added D4: TVS, Diode_SMD:D_0402_1005Metric, F.Cu at (22.9, -81.3)
- added D5: TVS, Diode_SMD:D_0402_1005Metric, F.Cu at (30.5, -80.7)
- added R32: 270, Resistor_SMD:R_0402_1005Metric, F.Cu at (12.4, -70.1)
- C1: value 10uF Tan. -> 10uF
- C4: value 1uF Tan. -> 1uF
- D28: value LG_R971-KN-1 -> LTST-C193KRKT-5A; footprint digikey-footprints:0805 -> LED_SMD:LED_0603_1608Metric
- moved TP12 314.9 mm to (5.59, -74.7), turned to 90 degrees
- moved TP10 313.1 mm to (29.4, -68.8), turned to 90 degrees
- moved R10 310.5 mm to (20.1, -79.0), turned to -90 degrees
- moved Q2 310.1 mm to (34.9, -79.5)
- moved R8 308.3 mm to (20.1, -76.7), turned to 90 degrees
- moved R6 306.1 mm to (20.1, -74.2), turned to 90 degrees
- moved U5 305.8 mm to (33.1, -75.1)
- moved C17 304.8 mm to (31.1, -66.5)
- moved R11 304.5 mm to (37.3, -70.1)
- moved R4 304.2 mm to (21.5, -72.9), turned to -90 degrees
- moved IC2 303.5 mm to (35.0, -67.3), turned to 180 degrees
- moved TP11 303.1 mm to (36.6, -63.7)
- moved C16 302.8 mm to (31.4, -71.5), turned to -90 degrees
- moved TP8 301.0 mm to (2.29, -73.2), turned to 90 degrees
- moved TP5 300.1 mm to (-4.57, -5.59)
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Connections:
- C12 pad 2: Net-(C12-Pad2) -> VBUS
- D28 pad 2: GND -> Net-(D28-Pad2)
- Q1 pad 2: Net-(C12-Pad2) -> VBUS
- TP7 pad 1: Net-(C12-Pad2) -> VBUS
- U4 pad 1: Net-(C12-Pad2) -> VBUS
Routing:
- net /USB and MCU LDO/BATT_IN_POS: track 0.00 -> 9.08 mm
- net Net-(R28-Pad2): track 0.00 -> 6.39 mm
- net Net-(IC1-Pad3): track 0.00 -> 5.32 mm
- net /USB and MCU LDO/IMON: track 0.00 -> 3.76 mm
- net Net-(IC1-Pad15): track 0.00 -> 3.49 mm
- net Net-(IC1-Pad14): track 0.00 -> 3.22 mm
- net Net-(L1-Pad1): track 0.00 -> 3.04 mm
- net /USB and MCU LDO/ILIM: track 0.00 -> 2.35 mm
- net Net-(C14-Pad1): track 0.00 -> 2.17 mm
- net Net-(R29-Pad2): track 0.00 -> 2.15 mm
- net Net-(C26-Pad1): track 1.06 -> 0.00 mm
- net /PR_EN: track 0.00 -> 0.88 mm, vias 0 -> 1
- net GND: vias 0 -> 18
- added copper zone on F.Cu, net /Passive Retainment/Burn_HS
- added copper zone on F.Cu, net /USB and MCU LDO/BATT_IN_POS
- added copper zone on F.Cu, net /USB and MCU LDO/LDO_IN
- added copper zone on F.Cu, net BATT +
- added copper zone on F.Cu, net GND
- added copper zone on In2.Cu, net GND
- added copper zone on F.Cu, net VBUS

Commit message: Layout rough draft
Parts:
- removed TP3, TP4: TestPoint, TestPoint:TestPoint_Pad_D1.0mm
- added J14: Conn_01x02, Connector_PinSocket_2.00mm:PinSocket_1x02_P2.00mm_Vertical, F.Cu at (66.1, -62.1)
- added J15: Conn_01x02, Connector_PinSocket_2.00mm:PinSocket_1x02_P2.00mm_Vertical, F.Cu at (64.1, -58.7)
- added S1: KSR253GLFG, Miles Added:KSR253GLFG, F.Cu at (71.7, -54.8)
- J1: value Headers -> Conn_02x08_Odd_Even; footprint Connector_PinSocket_2.00mm:PinSocket_2x30_P2.00mm_Vertical -> Connector_PinHeader_2.00mm:PinHeader_2x08_P2.00mm_Vertical
- J2: value Aux. Photodiode Board 1 -> 70543-0108; footprint Miles Added:1719730004 -> Miles Added:SHDR4W64P0X254_1X4_1271X508X1181P
- J3: value Aux. Photodiode Board 2 -> 70543-0108; footprint Miles Added:1719730004 -> Miles Added:SHDR4W64P0X254_1X4_1271X508X1181P
- J5: value Systems Board Connector -> 70543-0108; footprint Miles Added:1719730004 -> Miles Added:SHDR4W64P0X254_1X4_1271X508X1181P
- JP1: footprint Connector_PinHeader_2.00mm:PinHeader_1x03_P2.00mm_Vertical_SMD_Pin1Left -> Connector_PinHeader_2.00mm:PinHeader_1x03_P2.00mm_Vertical
- moved TP6 67.5 mm to (40.9, -45.7), turned to 90 degrees
- moved J6 67.2 mm to (39.9, -31.3), turned to 0 degrees
- moved C11 64.7 mm to (36.7, -43.5), turned to -90 degrees
- moved U3 64.7 mm to (37.4, -47.1)
- moved D8 62.1 mm to (38.9, -43.5), turned to -90 degrees
- moved C10 59.2 mm to (33.7, -45.3)
- moved R3 55.6 mm to (33.6, -43.3), turned to 180 degrees
- moved J1 55.3 mm to (25.2, -32.6)
- moved TP5 53.2 mm to (31.3, -44.9), turned to 90 degrees
- moved U2 45.1 mm to (31.2, -31.9)
- moved R1 33.6 mm to (63.6, -55.8), turned to -90 degrees
- moved R2 33.2 mm to (63.6, -53.0), turned to 90 degrees
- moved J3 33.0 mm to (64.5, -45.8)
- moved D7 32.9 mm to (61.7, -53.0), turned to -90 degrees
- moved J2 32.5 mm to (70.9, -39.3), turned to -90 degrees
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Connections:
- net /USB and MCU LDO/USB_CONN_DM renamed /USB and MCU LDO/USB_CONN_DN
- net Net-(J11-Pad2) renamed /Passive Retainment/Burn_LS
- J1 pad 1: /VDD -> +3V3
- J1 pad 10: /PR_EN -> unconnected-(J1-Pad10)
- J1 pad 11: /Burn_sig -> /SYS_SCL
- J1 pad 12: BATT + -> /Burn_sig
- J1 pad 13: BATT + -> /SYS_SDA
- J1 pad 14: /PA0 -> /PR_EN
- J1 pad 15: /PA1 -> BATT +
- J1 pad 16: /PA2 -> GND
- J1 pad 2: /PC13 (RTC) -> /PA7
- J1 pad 3: /PC14 (RTC) -> /PC15 (RTC)
- J1 pad 4: /PC15 (RTC) -> /PA6
- J1 pad 5: /OSC_IN -> /PC14 (RTC)
- J1 pad 6: /OSC_OUT -> unconnected-(J1-Pad6)
- J1 pad 7: /NRST -> /PC13 (RTC)
- J1 pad 8: /SYS_SCL -> unconnected-(J1-Pad8)
- J1 pad 9: /SYS_SDA -> unconnected-(J1-Pad9)
- J2 pad 3: +3V3 -> BATT +
- J3 pad 3: +3V3 -> BATT +
- U1 pad 11: /Burn_sig -> unconnected-(U1-Pad11)
- U1 pad 14: /PA0 -> unconnected-(U1-Pad14)
- U1 pad 15: /PA1 -> unconnected-(U1-Pad15)
- U1 pad 16: /PA2 -> unconnected-(U1-Pad16)
- U1 pad 17: /PA3 -> unconnected-(U1-Pad17)
- U1 pad 24: /PC4 -> unconnected-(U1-Pad24)
- U1 pad 33: /PB12 -> unconnected-(U1-Pad33)
- U1 pad 34: /PB13 -> unconnected-(U1-Pad34)
- U1 pad 35: /PB14 -> unconnected-(U1-Pad35)
- U1 pad 41: /PA8 -> unconnected-(U1-Pad41)
- U1 pad 42: /PA9 -> unconnected-(U1-Pad42)
- U1 pad 43: /PA10 -> unconnected-(U1-Pad43)
- U1 pad 44: /USB_OTG_FS_DM -> /USB_OTG_FS_DN
- U1 pad 51: /PC10 -> unconnected-(U1-Pad51)
- U1 pad 52: /PC11 -> unconnected-(U1-Pad52)
- U1 pad 53: /PC12 -> unconnected-(U1-Pad53)
- U1 pad 54: /PD2 -> /Burn_sig
- U11 pad 6: /USB_OTG_FS_DM -> /USB_OTG_FS_DN
Routing:
- net /SYS_SDA: track 0.00 -> 123.1 mm, vias 0 -> 4
- net /SYS_SCL: track 0.00 -> 118.0 mm, vias 0 -> 3
- net GND: track 0.00 -> 90.3 mm, vias 18 -> 156
- net /PA6: track 0.00 -> 70.8 mm
- net /PA7: track 0.00 -> 69.9 mm
- net /PR_EN: track 0.88 -> 69.2 mm, vias 1 -> 4
- net /Burn_sig: track 0.00 -> 65.9 mm, vias 0 -> 2
- net +3V3: track 0.00 -> 45.8 mm, vias 0 -> 18
- net /MUX (S0): track 0.00 -> 45.6 mm, vias 0 -> 2
- net /MUX (S1): track 0.00 -> 44.5 mm, vias 0 -> 2
- net /MUX (S2): track 0.00 -> 42.8 mm, vias 0 -> 2
- net /BOOT: track 0.00 -> 42.0 mm, vias 0 -> 1
- net /PC13 (RTC): track 0.00 -> 41.3 mm
- net /MTR2_STCK: track 0.00 -> 38.8 mm, vias 0 -> 2
- net /PC14 (RTC): track 0.00 -> 38.6 mm
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- added copper zone on F.Cu, net +3V3
- added copper zone on In2.Cu, net +3V3
- added copper zone on F.Cu, net /Passive Retainment/Burn_LS
- added copper zone on In2.Cu, net BATT +
- added copper zone on In1.Cu, net GND
- added copper zone on F.Cu, net Net-(C10-Pad2)
- removed copper zone on In2.Cu, net GND
Other:
- board size 83 x 83 mm -> 83 x 55 mm

Commit message: V1.0 Finished
Submitted to manufacturing.
Parts:
- added G***: LOGO, LOGO, F.Cu at (140.7, 117.5)
- added G***: LOGO, LOGO, B.Cu at (147.9, 95.7)
- moved C10 183.9 mm to (138.5, 105.9)
- moved C11 183.9 mm to (141.4, 107.6)
- moved C12 183.9 mm to (150.0, 77.3)
- moved C14 183.9 mm to (128.7, 78.2)
- moved C15 183.9 mm to (141.3, 77.3)
- moved C16 183.9 mm to (136.1, 81.1)
- moved C17 183.9 mm to (136.2, 87.2)
- moved C18 183.9 mm to (144.2, 86.1)
- moved C19 183.9 mm to (174.4, 78.0)
- moved C21 183.9 mm to (162.2, 71.7)
- moved C22 183.9 mm to (164.4, 79.5)
- moved C23 183.9 mm to (164.5, 75.2)
- moved C25 183.9 mm to (118.8, 92.6)
- moved C26 183.9 mm to (129.2, 95.8)
- moved C27 183.9 mm to (129.2, 87.0)
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Routing:
- net GND: track 90.3 -> 91.4 mm, vias 156 -> 143
- net /Burn_sig: track 65.9 -> 65.2 mm
- net /SYS_SCL: track 118.0 -> 118.7 mm
- net /PR_EN: track 69.2 -> 69.3 mm, vias 4 -> 5
- net /STEP_VREF2: vias 1 -> 0
- net /Passive Retainment/Burn_LS: vias 9 -> 0
Other:
- outline, holes or cut-outs redrawn
- board text added: "An."
- board text added: "Att. Det. PhDiodes 0 1 2 3 4 5 6 7"
- board text added: "B+"
- board text added: "BATT"
- board text added: "BOOT"
- board text added: "BURN+"
- board text added: "BURN-"
- board text added: "Cal Poly JUCI Team Solar Array Drive Assembly Board April 7, 2023 Ver. 1.0"
- board text added: "Cat."
- board text added: "DAC1"
- board text added: "DAC2"
- board text added: "GND"
- board text added: "Motor 1"
- board text added: "Motor 1: BLU RED GRN BLK"
- board text added: "Motor 2"
- board text added: "Motor 2: BLU RED GRN BLK"
- board text added: "NRST"
- board text added: "PB10"
- board text added: "PB11"
- board text added: "Passive Retainment"
- board text added: "SCL"
- board text added: "SDA"
- board text added: "Sun Sense 1"
- board text added: "Sun Sense 2"
- board text added: "Sys. Board"
