File: Electrical/SADA_Board/SADA_Board/Passive_retainment.kicad_sch (KiCad schematic)
At the start: 8 parts

Commit message: Pre-passive retainment change
Parts:
- added EXT?: NiCr Wire Connector, 0_custom:EXT_no_footprint, symbol 0_custom:{lt}name{gt}
Other:
- note added: "Buck regulator that can handle 4 amps?"
Changed lines of the file:
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@@
+    (effects (font (size 2 2)) (justify left bottom))
+  )
+  (text "Buck regulator that can handle 4 amps?" (at 125.349 58.42 0)
     (effects (font (size 2 2)) (justify left bottom))
   )
@@
     (pin "2")
   )
+  (symbol (lib_id "0_custom:{lt}name{gt}") (at 195.3604 134.0886 0) (unit 1)
+    (in_bom yes) (on_board yes) (fields_autoplaced)
+    (property "Reference" "EXT?" (id 0) (at 197.2654 132.8185 0)
+      (effects (font (size 1.27 1.27)) (justify left))
+    )
+    (property "Value" "NiCr Wire Connector" (id 1) (at 197.2654 135.3585 0)
+      (effects (font (size 1.27 1.27)) (justify left))
+    )
+    (property "Footprint" "0_custom:EXT_no_footprint" (id 2) (at 195.3604 134.0886 0)
+      (effects (font (size 1.27 1.27)) hide)
+    )
+    (property "Datasheet" "" (id 3) (at 195.3604 134.0886 0)
+      (effects (font (size 1.27 1.27)) hide)
+    )
+    (property "MPN" "3-640427-2" (id 4) (at 195.3604 134.0886 0)
+      (effects (font (size 1.27 1.27)) hide)
+    )
+  )
   (symbol (lib_id "Device:C") (at 80.391 103.759 0) (unit 1)

Commit message: pre-gio review
Parts:
- removed C?: 4.7uF Cer., Capacitor_SMD:C_0603_1608Metric, symbol Device:C
- removed C?: 2.2uF Cer., Capacitor_SMD:C_0603_1608Metric, symbol Device:C
- removed R?: 47k, Resistor_SMD:R_0603_1608Metric, symbol Device:R_US
- removed R?: 7.5k, Resistor_SMD:R_0603_1608Metric_Pad0.98x0.95mm_HandSolder, symbol Device:R_US
- removed R?: 15k, Resistor_SMD:R_0603_1608Metric, symbol Device:R_US
- removed U?: XC6230A001QR-G, SOIC127P600X175-9N, symbol XC6230A001QR-G:XC6230A001QR-G
- added C29, C30: 10uF, Capacitor_SMD:C_0603_1608Metric, symbol Device:C
- added C31, C32: 22 uF, Capacitor_SMD:C_1210_3225Metric, symbol Device:C
- added D10, D11, D12, D13: TVS, symbol Diode:ESD5Zxx
- added EXT11: NiCr Wire Connector, 0_custom:EXT_no_footprint, symbol 0_custom:{lt}name{gt}
- added J12: 105431-1202, Miles Added:1054311202, symbol molex_105431-1202:105431-1202
- added L1: 220 nH, Miles Added:INDPM3630X150N, symbol IHLP1212AEERR22M11:IHLP1212AEERR22M11
- added R28: 200k, Resistor_SMD:R_0603_1608Metric_Pad0.98x0.95mm_HandSolder, symbol Device:R_US
- added R29, R30: 100k, Resistor_SMD:R_0402_1005Metric, symbol Device:R_US
- added TP22: TestPoint, TestPoint:TestPoint_Pad_D1.5mm, symbol Connector:TestPoint
- added U10: Si1442DH, Package_TO_SOT_SMD:SOT-363_SC-70-6, symbol 0_custom:Si1442DH
- added U8: TPS62867RQYR, 0_custom:VQFN-9, symbol 0_custom:TPS62867RQYR
- gave numbers to parts that had none: 3
Connections:
- net BATT +: now also C29.2, C30.1, D11.1 (K), R29.1, U8.3 (V_IN)
- net Burn_sig: now also U10.3 (G)
- net GND: now also C29.1, C30.2, C31.1, C32.2, D10.2 (A), D11.2 (A), D12.2 (A), D13.2 (A), J12.MP1, J12.MP2, R30.2, U10.4 (S), U8.1 (AGND), U8.2 (PGND), U8.6 (VSET/MODE)
- net NiCr_HS renamed Burn_HS
- net Burn_HS: now also C31.2, C32.1, D10.1 (K), J12.1, L1.2, R28.1, TP22.1, U8.8 (VOS)
- net NiCr_LS: no longer names the net of J11.2, U9.1 (D), U9.2 (D), U9.5 (D), U9.6 (D)
- net NiCr_LS: now also D12.1 (K)
- new net: D13.1 (K), J12.2, U10.1 (D), U10.2 (D), U10.5 (D), U10.6 (D)
- new net: R28.2, R30.1, U8.9 (FB)
- new net: R29.2, U8.5 (PG)
- new net: L1.1, U8.7 (SW)
- new net PR_EN: U8.4 (EN)
- no-connect marks 1 -> 0
Other:
- note removed: "Buck regulator that can handle 4 amps?"
- title: (none) -> PASSIVE RETAINMENT
- moved on the sheet: EXT10, J11, U9

Commit message: ESD changes
Parts:
- removed D12, D13: TVS, symbol Diode:ESD5Zxx
- removed EXT11: NiCr Wire Connector, 0_custom:EXT_no_footprint, symbol 0_custom:{lt}name{gt}
- removed J12: 105431-1202, Miles Added:1054311202, symbol molex_105431-1202:105431-1202
- removed U10, U9: Si1442DH, Package_TO_SOT_SMD:SOT-363_SC-70-6, symbol 0_custom:Si1442DH
- added Q3: IRLML6244TRPBF, SOT95P237X112-3N, symbol IRLML6244TRPBF:IRLML6244TRPBF
- D10, D11: footprint (none) -> Diode_SMD:D_0402_1005Metric
- TP22: footprint TestPoint:TestPoint_Pad_D1.5mm -> TestPoint:TestPoint_Pad_D1.0mm
Connections:
- net Burn_sig: now also Q3.1 (G)
- net GND: now also Q3.2 (S)
- net at J11.2: now also Q3.3 (D)

Commit message: Layout rough draft
Connections:
- net Burn_LS: now reaches J11.2, Q3.3 (D)
Changed lines of the file:
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@@
     (effects (font (size 2 2)) (justify left bottom))
+  )
+  (label "Burn_LS" (at 215.6627 77.3938 0)
+    (effects (font (size 1.27 1.27)) (justify left bottom))
   )
   (label "Burn_HS" (at 215.6206 74.8538 0)

Commit message: Updated BOM
Parts:
- D10, D11: MPN (none) -> ESD321DPYR
- EXT10: value NiCr Wire Connector -> Power Male Connector
- J11: MPN (none) -> 105431-1202; Manufacturer_Part_Number 105431-1202 -> (none)
- L1: MPN (none) -> IHLP1212AEERR22M11; Manufacturer_Part_Number IHLP1212AEERR22M11 -> (none)
- Q3: MPN (none) -> IRLML6244TRPBF; Manufacturer_Part_Number IRLML6244TRPBF -> (none)
- TP22: now left out of the parts list
Other:
- company: (none) -> Cal Poly, SLO
- title: PASSIVE RETAINMENT -> CubeSat SADA - Main
Changed lines of the file:
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@@
   (paper "A4")
   (title_block
-    (title "PASSIVE RETAINMENT")
+    (title "CubeSat SADA - Main")
+    (date "2023-04-07")
+    (rev "V1.0")
+    (company "Cal Poly, SLO")
   )
   (junction (at 141.986 71.12) (diameter 0) (color 0 0 0 0)
@@
       (effects (font (size 1.27 1.27)) (justify left) hide)
     )
-    (property "Manufacturer_Part_Number" "IRLML6244TRPBF" (id 9) (at 204.47 98.552 0)
+    (property "MPN" "IRLML6244TRPBF" (id 9) (at 204.47 98.552 0)
       (effects (font (size 1.27 1.27)) (justify left) hide)
     )
@@
       (effects (font (size 1.27 1.27)) hide)
     )
-    (property "MPN" "" (id 4) (at 186.436 65.278 0)
+    (property "MPN" "ESD321DPYR" (id 4) (at 186.436 65.278 0)
       (effects (font (size 1.27 1.27)) hide)
     )
@@
       (effects (font (size 1.27 1.27)) (justify left) hide)
     )
-    (property "Manufacturer_Part_Number" "105431-1202" (id 9) (at 247.3706 64.6938 0)
+    (property "MPN" "105431-1202" (id 9) (at 247.3706 64.6938 0)
       (effects (font (size 1.27 1.27)) (justify left) hide)
     )
@@
       (effects (font (size 1.27 1.27)) (justify left))
     )
-    (property "Value" "NiCr Wire Connector" (id 1) (at 231.2416 89.8397 0)
+    (property "Value" "Power Male Connector" (id 1) (at 231.2416 89.8397 0)
       (effects (font (size 1.27 1.27)) (justify left))
     )
@@
       (effects (font (size 1.27 1.27)) (justify left) hide)
     )
-    (property "Manufacturer_Part_Number" "IHLP1212AEERR22M11" (id 9) (at 135.128 87.63 0)
+    (property "MPN" "IHLP1212AEERR22M11" (id 9) (at 135.128 87.63 0)
       (effects (font (size 1.27 1.27)) (justify left) hide)
     )
@@
       (effects (font (size 1.27 1.27)) hide)
     )
-    (property "MPN" "" (id 4) (at 74.93 67.31 0)
+    (property "MPN" "ESD321DPYR" (id 4) (at 74.93 67.31 0)
       (effects (font (size 1.27 1.27)) hide)
     )
@@
   )
   (symbol (lib_id "Connector:TestPoint") (at 161.7072 71.0438 0) (unit 1)
-    (in_bom yes) (on_board yes) (fields_autoplaced)
+    (in_bom no) (on_board yes) (fields_autoplaced)
     (property "Reference" "TP22" (id 0) (at 163.7392 67.7417 0)
       (effects (font (size 1.27 1.27)) (justify left))
