File: Electrical/SADA_Board/SADA_Board/Bipolar_Steppers.kicad_sch (KiCad schematic)
At the start: 32 parts, among them J15 171973-0004, J16 171973-0004, U10 STSPIN220, U9 STSPIN220

Commit message: pre-gio review
Parts:
- added D14, D15, D16, D17, D18, D19, D20, D21, D22, D23, D24, D25, D26, D27: TVS, symbol Diode:ESD5Zxx
- added TP13, TP14, TP15, TP16, TP17, TP18, TP19, TP20, TP21: TestPoint, TestPoint:TestPoint_Pad_D1.5mm, symbol Connector:TestPoint
- renumbered C20 to C19, C21 to C20, C22 to C21, C23 to C22, C24 to C23, C25 to C24, C26 to C25, C27 to C26, C28 to C27, C29 to C28, EXT13 to EXT8, EXT14 to EXT9, J16 to J10, J15 to J9, R24 to R12, R25 to R13, R26 to R14, R27 to R15, R28 to R16, R29 to R17, R30 to R18, R31 to R19, R32 to R20, R33 to R21, R34 to R22, R35 to R23, R36 to R24, R37 to R25, R38 to R26, R39 to R27, U9 to U6, U10 to U7
Connections:
- net BATT +: now also D14.1 (K), D21.1 (K)
- net GND: now also D14.2 (A), D15.2 (A), D16.2 (A), D17.2 (A), D18.2 (A), D19.2 (A), D20.2 (A), D21.2 (A), D22.2 (A), D23.2 (A), D24.2 (A), D25.2 (A), D26.2 (A), D27.2 (A)
- net MTR1_BLK: now also TP14.1
- net MTR1_BLU: now also TP19.1
- net MTR1_DIR: now also D16.1 (K), TP13.1
- net MTR1_FAULT: no longer U7.13 (EN/FLT)
- net MTR1_GRN: now also TP16.1
- net MTR1_RED: now also TP18.1
- net MTR1_STBY: now also D17.1 (K); no longer U7.14 (STBY/RESET)
- net MTR1_STCK: now also D15.1 (K), TP15.1
- net MTR2_DIR: now also D23.1 (K)
- net MTR2_FAULT: now also U7.13 (EN/FLT), D25.1 (K)
- net MTR2_STBY: now also U7.14 (STBY/RESET), D24.1 (K)
- net MTR2_STCK: now also D22.1 (K)
- net SENSE_A_M1: now also TP17.1
- net SENSE_B_M1: now also TP20.1
- net T_OFF_1: now also D20.1 (K)
- net T_OFF_2: now also D26.1 (K)
- net V_REF1: now also D19.1 (K), TP21.1
- net V_REF2: now also D27.1 (K)
Other:
- note added: "Identical Frequency- Necessary to ensure identical movement?"
- moved on the sheet: J9, R24, R25

Commit message: ESD changes
Parts:
- D14, D15, D16, D17, D18, D19, D20, D21, D22, D23, D24, D25, D26, D27: footprint (none) -> Diode_SMD:D_0402_1005Metric
- TP13, TP14, TP15, TP16, TP17, TP18, TP19, TP20, TP21: footprint TestPoint:TestPoint_Pad_D1.5mm -> TestPoint:TestPoint_Pad_D1.0mm
Changed lines of the file:
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@@
       (effects (font (size 1.27 1.27)) (justify right) hide)
     )
-    (property "Footprint" "TestPoint:TestPoint_Pad_D1.5mm" (id 2) (at 188.976 68.58 0)
+    (property "Footprint" "TestPoint:TestPoint_Pad_D1.0mm" (id 2) (at 188.976 68.58 0)
       (effects (font (size 1.27 1.27)) hide)
     )
@@
       (effects (font (size 1.27 1.27)) hide)
     )
-    (property "Footprint" "" (id 2) (at 161.417 70.358 0)
+    (property "Footprint" "Diode_SMD:D_0402_1005Metric" (id 2) (at 161.417 70.358 0)
       (effects (font (size 1.27 1.27)) hide)
     )
@@
       (effects (font (size 1.27 1.27)) hide)
     )
-    (property "Footprint" "" (id 2) (at 163.068 109.855 0)
+    (property "Footprint" "Diode_SMD:D_0402_1005Metric" (id 2) (at 163.068 109.855 0)
       (effects (font (size 1.27 1.27)) hide)
     )
@@
       (effects (font (size 1.27 1.27)) hide)
     )
-    (property "Footprint" "" (id 2) (at 208.026 33.655 0)
+    (property "Footprint" "Diode_SMD:D_0402_1005Metric" (id 2) (at 208.026 33.655 0)
       (effects (font (size 1.27 1.27)) hide)
     )
@@
       (effects (font (size 1.27 1.27)) (justify right) hide)
     )
-    (property "Footprint" "TestPoint:TestPoint_Pad_D1.5mm" (id 2) (at 173.99 48.26 0)
+    (property "Footprint" "TestPoint:TestPoint_Pad_D1.0mm" (id 2) (at 173.99 48.26 0)
       (effects (font (size 1.27 1.27)) hide)
     )
@@
       (effects (font (size 1.27 1.27)) hide)
     )
-    (property "Footprint" "" (id 2) (at 163.703 147.32 0)
+    (property "Footprint" "Diode_SMD:D_0402_1005Metric" (id 2) (at 163.703 147.32 0)
       (effects (font (size 1.27 1.27)) hide)
     )
@@
       (effects (font (size 1.27 1.27)) hide)
     )
-    (property "Footprint" "" (id 2) (at 208.153 110.617 0)
+    (property "Footprint" "Diode_SMD:D_0402_1005Metric" (id 2) (at 208.153 110.617 0)
       (effects (font (size 1.27 1.27)) hide)
     )
@@
       (effects (font (size 1.27 1.27)) hide)
     )
-    (property "Footprint" "" (id 2) (at 179.451 77.978 0)
+    (property "Footprint" "Diode_SMD:D_0402_1005Metric" (id 2) (at 179.451 77.978 0)
       (effects (font (size 1.27 1.27)) hide)
     )
@@
       (effects (font (size 1.27 1.27)) hide)
     )
-    (property "Footprint" "" (id 2) (at 183.261 77.978 0)
+    (property "Footprint" "Diode_SMD:D_0402_1005Metric" (id 2) (at 183.261 77.978 0)
       (effects (font (size 1.27 1.27)) hide)
     )
@@
       (effects (font (size 1.27 1.27)) hide)
     )
-    (property "Footprint" "" (id 2) (at 167.513 147.32 0)
+    (property "Footprint" "Diode_SMD:D_0402_1005Metric" (id 2) (at 167.513 147.32 0)
       (effects (font (size 1.27 1.27)) hide)
     )
@@
       (effects (font (size 1.27 1.27)) hide)
     )
-    (property "Footprint" "" (id 2) (at 159.766 36.703 0)
+    (property "Footprint" "Diode_SMD:D_0402_1005Metric" (id 2) (at 159.766 36.703 0)
       (effects (font (size 1.27 1.27)) hide)
     )
@@
       (effects (font (size 1.27 1.27)) hide)
     )
-    (property "Footprint" "" (id 2) (at 163.068 113.665 0)
+    (property "Footprint" "Diode_SMD:D_0402_1005Metric" (id 2) (at 163.068 113.665 0)
       (effects (font (size 1.27 1.27)) hide)
     )
@@
       (effects (font (size 1.27 1.27)) (justify right) hide)
     )
-    (property "Footprint" "TestPoint:TestPoint_Pad_D1.5mm" (id 2) (at 229.362 63.5 0)
+    (property "Footprint" "TestPoint:TestPoint_Pad_D1.0mm" (id 2) (at 229.362 63.5 0)
       (effects (font (size 1.27 1.27)) hide)
     )
@@
       (effects (font (size 1.27 1.27)) hide)
     )
-    (property "Footprint" "" (id 2) (at 180.975 154.94 0)
+    (property "Footprint" "Diode_SMD:D_0402_1005Metric" (id 2) (at 180.975 154.94 0)
       (effects (font (size 1.27 1.27)) hide)
     )
@@
       (effects (font (size 1.27 1.27)) hide)
     )
-    (property "Footprint" "" (id 2) (at 174.879 154.94 0)
+    (property "Footprint" "Diode_SMD:D_0402_1005Metric" (id 2) (at 174.879 154.94 0)
       (effects (font (size 1.27 1.27)) hide)
     )
@@
       (effects (font (size 1.27 1.27)) (justify right) hide)
     )
-    (property "Footprint" "TestPoint:TestPoint_Pad_D1.5mm" (id 2) (at 229.362 68.58 0)
+    (property "Footprint" "TestPoint:TestPoint_Pad_D1.0mm" (id 2) (at 229.362 68.58 0)
       (effects (font (size 1.27 1.27)) hide)
     )
@@
       (effects (font (size 1.27 1.27)) (justify right) hide)
     )
-    (property "Footprint" "TestPoint:TestPoint_Pad_D1.5mm" (id 2) (at 229.362 66.04 0)
+    (property "Footprint" "TestPoint:TestPoint_Pad_D1.0mm" (id 2) (at 229.362 66.04 0)
       (effects (font (size 1.27 1.27)) hide)
     )
@@
       (effects (font (size 1.27 1.27)) hide)
     )
-    (property "Footprint" "" (id 2) (at 159.766 32.893 0)
+    (property "Footprint" "Diode_SMD:D_0402_1005Metric" (id 2) (at 159.766 32.893 0)
       (effects (font (size 1.27 1.27)) hide)
     )
@@
       (effects (font (size 1.27 1.27)) (justify right) hide)
     )
-    (property "Footprint" "TestPoint:TestPoint_Pad_D1.5mm" (id 2) (at 229.87 53.34 0)
+    (property "Footprint" "TestPoint:TestPoint_Pad_D1.0mm" (id 2) (at 229.87 53.34 0)
       (effects (font (size 1.27 1.27)) hide)
     )
@@
       (effects (font (size 1.27 1.27)) (justify right) hide)
     )
-    (property "Footprint" "TestPoint:TestPoint_Pad_D1.5mm" (id 2) (at 184.15 45.72 0)
+    (property "Footprint" "TestPoint:TestPoint_Pad_D1.0mm" (id 2) (at 184.15 45.72 0)
       (effects (font (size 1.27 1.27)) hide)
     )
@@
       (effects (font (size 1.27 1.27)) (justify right) hide)
     )
-    (property "Footprint" "TestPoint:TestPoint_Pad_D1.5mm" (id 2) (at 229.87 50.8 0)
+    (property "Footprint" "TestPoint:TestPoint_Pad_D1.0mm" (id 2) (at 229.87 50.8 0)
       (effects (font (size 1.27 1.27)) hide)
     )
@@
       (effects (font (size 1.27 1.27)) hide)
     )
-    (property "Footprint" "" (id 2) (at 157.607 70.358 0)
+    (property "Footprint" "Diode_SMD:D_0402_1005Metric" (id 2) (at 157.607 70.358 0)
       (effects (font (size 1.27 1.27)) hide)
     )
@@
       (effects (font (size 1.27 1.27)) (justify right) hide)
     )
-    (property "Footprint" "TestPoint:TestPoint_Pad_D1.5mm" (id 2) (at 229.87 55.88 0)
-      (effects (font (size 1.27 1.27)) hide)
-    )
+    (property "Footprint" "TestPoint:TestPoint_Pad_D1.0mm" (id 2) (at 229.87 55.88 0)
+      (effects (font (size 1.27 1.27)) hide)
+    )

Commit message: layout prog
Connections:
- net MTR1_FAULT: now also D18.1 (K)
Changed lines of the file:
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@@
   (junction (at 201.295 155.702) (diameter 0) (color 0 0 0 0)
   )
+  (junction (at 165.862 60.96) (diameter 0) (color 0 0 0 0)
+  )
   (junction (at 201.295 106.172) (diameter 0) (color 0 0 0 0)
   )
@@
   (junction (at 183.896 68.58) (diameter 0) (color 0 0 0 0)
   )
-  (junction (at 165.8671 60.9599) (diameter 0) (color 0 0 0 0)
-  )
   (junction (at 144.145 126.365) (diameter 0) (color 0 0 0 0)
   )
@@
     (stroke (width 0) (type default) (color 0 0 0 0))
   )
-  (wire (pts (xy 165.8671 60.9599) (xy 165.862 66.548))
-    (stroke (width 0) (type default) (color 0 0 0 0))
-  )
   (wire (pts (xy 34.925 31.75) (xy 34.925 38.1))
     (stroke (width 0) (type default) (color 0 0 0 0))
@@
     (stroke (width 0) (type default) (color 0 0 0 0))
   )
-  (wire (pts (xy 160.782 60.96) (xy 188.595 60.96))
+  (wire (pts (xy 160.782 60.96) (xy 165.862 60.96))
     (stroke (width 0) (type default) (color 0 0 0 0))
   )
@@
     (stroke (width 0) (type default) (color 0 0 0 0))
   )
+  (wire (pts (xy 165.862 60.96) (xy 165.862 66.548))
+    (stroke (width 0) (type default) (color 0 0 0 0))
+  )
   (wire (pts (xy 129.54 126.365) (xy 132.715 126.365))
     (stroke (width 0) (type default) (color 0 0 0 0))
@@
     (stroke (width 0) (type default) (color 0 0 0 0))
   )
+  (wire (pts (xy 165.862 60.96) (xy 188.595 60.96))
+    (stroke (width 0) (type default) (color 0 0 0 0))
+  )

Commit message: Updated BOM
Parts:
- D14, D15, D16, D17, D18, D19, D20, D21, D22, D23, D24, D25, D26, D27: MPN (none) -> ESD321DPYR
- EXT8, EXT9: value Male MTR Conn. -> Male Conn.
- J10, J9: MPN (none) -> 171973-0004; Manufacturer_Part_Number 171973-0004 -> (none)
Other:
- company: (none) -> Cal Poly, SLO
- title: (none) -> CubeSat SADA - Main
Changed lines of the file:
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@@
 (kicad_sch (version 20211123) (generator eeschema)
   (paper "A4")
+  (title_block
+    (title "CubeSat SADA - Main")
+    (date "2023-04-07")
+    (rev "V1.0")
+    (company "Cal Poly, SLO")
+  )
   (junction (at 178.816 125.222) (diameter 0) (color 0 0 0 0)
   )
@@
   (symbol (lib_id "Diode:ESD5Zxx") (at 165.862 70.358 270) (unit 1)
     (in_bom yes) (on_board yes)
-    (property "Reference" "D18" (id 0) (at 168.91 73.914 90)
+    (property "Reference" "D18" (id 0) (at 171.45 70.358 90)
       (effects (font (size 1.27 1.27)) (justify right))
     )
@@
       (effects (font (size 1.27 1.27)) hide)
     )
-    (property "MPN" "" (id 4) (at 165.862 70.358 0)
+    (property "MPN" "ESD321DPYR" (id 4) (at 165.862 70.358 0)
       (effects (font (size 1.27 1.27)) hide)
     )
@@
   )
   (symbol (lib_id "Diode:ESD5Zxx") (at 163.068 114.3 180) (unit 1)
-    (in_bom yes) (on_board yes) (fields_autoplaced)
-    (property "Reference" "D22" (id 0) (at 163.0679 111.506 90)
+    (in_bom yes) (on_board yes)
+    (property "Reference" "D22" (id 0) (at 165.1 113.03 0)
       (effects (font (size 1.27 1.27)) (justify right))
     )
@@
       (effects (font (size 1.27 1.27)) hide)
     )
-    (property "MPN" "" (id 4) (at 163.068 114.3 0)
+    (property "MPN" "ESD321DPYR" (id 4) (at 163.068 114.3 0)
       (effects (font (size 1.27 1.27)) hide)
     )
@@
   )
   (symbol (lib_id "power:GND") (at 157.226 118.11 270) (unit 1)
-    (in_bom yes) (on_board yes) (fields_autoplaced)
+    (in_bom yes) (on_board yes)
     (property "Reference" "#PWR0112" (id 0) (at 150.876 118.11 0)
       (effects (font (size 1.27 1.27)) hide)
     )
-    (property "Value" "GND" (id 1) (at 152.4 118.11 0))
+    (property "Value" "GND" (id 1) (at 152.4 118.11 90))
     (property "Footprint" "" (id 2) (at 157.226 118.11 0)
       (effects (font (size 1.27 1.27)) hide)
@@
       (effects (font (size 1.27 1.27)) (justify left) hide)
     )
-    (property "Manufacturer_Part_Number" "171973-0004" (id 9) (at 263.525 147.32 0)
+    (property "MPN" "171973-0004" (id 9) (at 263.525 147.32 0)
       (effects (font (size 1.27 1.27)) (justify left) hide)
     )
@@
       (effects (font (size 1.27 1.27)) hide)
     )
-    (property "MPN" "" (id 4) (at 208.026 29.21 0)
+    (property "MPN" "ESD321DPYR" (id 4) (at 208.026 29.21 0)
       (effects (font (size 1.27 1.27)) hide)
     )
@@
       (effects (font (size 1.27 1.27)) hide)
     )
-    (property "MPN" "" (id 4) (at 168.148 147.32 0)
+    (property "MPN" "ESD321DPYR" (id 4) (at 168.148 147.32 0)
       (effects (font (size 1.27 1.27)) hide)
     )
@@
   )
   (symbol (lib_id "power:GND") (at 157.226 114.3 270) (unit 1)
-    (in_bom yes) (on_board yes) (fields_autoplaced)
+    (in_bom yes) (on_board yes)
     (property "Reference" "#PWR0111" (id 0) (at 150.876 114.3 0)
       (effects (font (size 1.27 1.27)) hide)
     )
-    (property "Value" "GND" (id 1) (at 152.4 114.3 0))
+    (property "Value" "GND" (id 1) (at 152.4 114.3 90))
     (property "Footprint" "" (id 2) (at 157.226 114.3 0)
       (effects (font (size 1.27 1.27)) hide)
@@
       (effects (font (size 1.27 1.27)) hide)
     )
-    (property "Value" "GND" (id 1) (at 171.958 157.988 0))
+    (property "Value" "GND" (id 1) (at 171.958 157.988 0)
+      (effects (font (size 1.27 1.27)) hide)
+    )
     (property "Footprint" "" (id 2) (at 171.958 153.162 0)
       (effects (font (size 1.27 1.27)) hide)
@@
       (effects (font (size 1.27 1.27)) hide)
     )
-    (property "MPN" "" (id 4) (at 208.153 106.172 0)
+    (property "MPN" "ESD321DPYR" (id 4) (at 208.153 106.172 0)
       (effects (font (size 1.27 1.27)) hide)
     )
@@
       (effects (font (size 1.27 1.27)) hide)
     )
-    (property "MPN" "" (id 4) (at 183.896 77.978 0)
+    (property "MPN" "ESD321DPYR" (id 4) (at 183.896 77.978 0)
       (effects (font (size 1.27 1.27)) hide)
     )
@@
   (symbol (lib_id "Diode:ESD5Zxx") (at 187.706 77.978 270) (unit 1)
     (in_bom yes) (on_board yes)
-    (property "Reference" "D20" (id 0) (at 190.754 81.026 90)
+    (property "Reference" "D20" (id 0) (at 193.548 77.978 90)
       (effects (font (size 1.27 1.27)) (justify right))
     )
@@
       (effects (font (size 1.27 1.27)) hide)
     )
-    (property "MPN" "" (id 4) (at 187.706 77.978 0)
+    (property "MPN" "ESD321DPYR" (id 4) (at 187.706 77.978 0)
       (effects (font (size 1.27 1.27)) hide)
     )
@@
       (effects (font (size 1.27 1.27)) (justify left))
     )
-    (property "Value" "Male MTR Conn." (id 1) (at 262.89 144.0179 0)
+    (property "Value" "Male Conn." (id 1) (at 262.89 144.0179 0)
       (effects (font (size 1.27 1.27)) (justify left))
     )
@@
   (symbol (lib_id "Diode:ESD5Zxx") (at 171.958 147.32 270) (unit 1)
     (in_bom yes) (on_board yes)
-    (property "Reference" "D25" (id 0) (at 175.006 150.876 90)
+    (property "Reference" "D25" (id 0) (at 176.022 150.114 90)
       (effects (font (size 1.27 1.27)) (justify right))
     )
@@
       (effects (font (size 1.27 1.27)) hide)
     )
-    (property "MPN" "" (id 4) (at 171.958 147.32 0)
+    (property "MPN" "ESD321DPYR" (id 4) (at 171.958 147.32 0)
       (effects (font (size 1.27 1.27)) hide)
     )
@@
       (effects (font (size 1.27 1.27)) hide)
     )
-    (property "MPN" "" (id 4) (at 159.766 41.148 0)
+    (property "MPN" "ESD321DPYR" (id 4) (at 159.766 41.148 0)
       (effects (font (size 1.27 1.27)) hide)
     )
@@
   (symbol (lib_id "Diode:ESD5Zxx") (at 163.068 118.11 180) (unit 1)
     (in_bom yes) (on_board yes)
-    (property "Reference" "D23" (id 0) (at 160.274 121.412 90)
+    (property "Reference" "D23" (id 0) (at 165.1 119.634 0)
       (effects (font (size 1.27 1.27)) (justify right))
     )
@@
       (effects (font (size 1.27 1.27)) hide)
     )
-    (property "MPN" "" (id 4) (at 163.068 118.11 0)
+    (property "MPN" "ESD321DPYR" (id 4) (at 163.068 118.11 0)
       (effects (font (size 1.27 1.27)) hide)
     )
@@
   )
   (symbol (lib_id "power:GND") (at 179.324 159.258 0) (unit 1)
-    (in_bom yes) (on_board yes) (fields_autoplaced)
+    (in_bom yes) (on_board yes)
     (property "Reference" "#PWR0115" (id 0) (at 179.324 165.608 0)
       (effects (font (size 1.27 1.27)) hide)
     )
-    (property "Value" "GND" (id 1) (at 179.324 164.084 0))
+    (property "Value" "GND" (id 1) (at 182.372 159.766 0))
     (property "Footprint" "" (id 2) (at 179.324 159.258 0)
       (effects (font (size 1.27 1.27)) hide)
@@
   )
   (symbol (lib_id "Diode:ESD5Zxx") (at 185.42 154.94 270) (unit 1)
-    (in_bom yes) (on_board yes) (fields_autoplaced)
-    (property "Reference" "D27" (id 0) (at 182.626 154.9401 90)
+    (in_bom yes) (on_board yes)
+    (property "Reference" "D27" (id 0) (at 191.262 155.194 90)
       (effects (font (size 1.27 1.27)) (justify right))
     )
@@
       (effects (font (size 1.27 1.27)) hide)
     )
-    (property "MPN" "" (id 4) (at 185.42 154.94 0)
+    (property "MPN" "ESD321DPYR" (id 4) (at 185.42 154.94 0)
       (effects (font (size 1.27 1.27)) hide)
     )
@@
   )
   (symbol (lib_id "Diode:ESD5Zxx") (at 179.324 154.94 270) (unit 1)
-    (in_bom yes) (on_board yes) (fields_autoplaced)
-    (property "Reference" "D26" (id 0) (at 176.53 154.9401 90)
+    (in_bom yes) (on_board yes)
+    (property "Reference" "D26" (id 0) (at 177.546 154.94 90)
       (effects (font (size 1.27 1.27)) (justify right))
     )
@@
       (effects (font (size 1.27 1.27)) hide)
     )
-    (property "MPN" "" (id 4) (at 179.324 154.94 0)
+    (property "MPN" "ESD321DPYR" (id 4) (at 179.324 154.94 0)
       (effects (font (size 1.27 1.27)) hide)
     )
@@
       (effects (font (size 1.27 1.27)) (justify left))
     )
-    (property "Value" "Male MTR Conn." (id 1) (at 262.89 66.0399 0)
+    (property "Value" "Male Conn." (id 1) (at 262.89 66.0399 0)
       (effects (font (size 1.27 1.27)) (justify left))
     )
@@
       (effects (font (size 1.27 1.27)) hide)
     )
-    (property "MPN" "" (id 4) (at 159.766 37.338 0)
+    (property "MPN" "ESD321DPYR" (id 4) (at 159.766 37.338 0)
       (effects (font (size 1.27 1.27)) hide)
     )
@@
       (effects (font (size 1.27 1.27)) hide)
     )
-    (property "Value" "GND" (id 1) (at 185.42 164.084 0))
+    (property "Value" "GND" (id 1) (at 185.42 164.084 0)
+      (effects (font (size 1.27 1.27)) hide)
+    )
     (property "Footprint" "" (id 2) (at 185.42 159.258 0)
       (effects (font (size 1.27 1.27)) hide)
@@
       (effects (font (size 1.27 1.27)) (justify left) hide)
     )
-    (property "Manufacturer_Part_Number" "171973-0004" (id 9) (at 266.192 68.58 0)
+    (property "MPN" "171973-0004" (id 9) (at 266.192 68.58 0)
       (effects (font (size 1.27 1.27)) (justify left) hide)
     )
@@
   )
   (symbol (lib_id "power:GND") (at 168.148 153.162 0) (unit 1)
-    (in_bom yes) (on_board yes) (fields_autoplaced)
+    (in_bom yes) (on_board yes)
     (property "Reference" "#PWR0113" (id 0) (at 168.148 159.512 0)
       (effects (font (size 1.27 1.27)) hide)
     )
-    (property "Value" "GND" (id 1) (at 168.148 157.988 0))
+    (property "Value" "GND" (id 1) (at 170.18 157.226 0))
     (property "Footprint" "" (id 2) (at 168.148 153.162 0)
       (effects (font (size 1.27 1.27)) hide)
@@
       (effects (font (size 1.27 1.27)) hide)
     )
-    (property "MPN" "" (id 4) (at 162.052 70.358 0)
-      (effects (font (size 1.27 1.27)) hide)
-    )
+    (property "MPN" "ESD321DPYR" (id 4) (at 162.052 70.358 0)
+      (effects (font (size 1.27 1.27)) hide)
+    )

Commit message: Upd. Schem and Datasheets
Other:
- note added: "SCHEMATIC NOTES - Designed for use with Pololu SY20STH30-0604A - Chosen to use EN pullup instead of MCU enable control - MODE1 and MODE2 grounded since only full stepping is used - Vref/RSNS chosen for max current of 0.6A/phase, though this is likely more current than necessary. R_SNS and V_ref can be changed if only significantly lower current is used - Vref set at constant 0.19 volts since no m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"
- note removed: "SCHEMATIC NOTES - Designed for use with Polalu S20STH30-0604A - Chosen to use EN pullup instead of MCU enable control - MODE1 and MODE2 grounded since only full stepping is used - Vref/RSNS chosen for max current of 0.6A/phase, though this is likely more current than necessary. R_SNS and V_ref can be changed if only significantly lower current is used - Vref set at constant 0.19 volts since no mi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"
Changed lines of the file:
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@@
     (effects (font (size 1.5 1.5)) (justify left bottom))
   )
-  (text "SCHEMATIC NOTES\n- Designed for use with Polalu S20STH30-0604A\n- Chosen to use EN pullup instead of MCU enable control\n- MODE1 and MODE2 grounded since only full stepping is used\n- Vref/RSNS chosen for max current of 0.6A/phase, though this is\n	likely more current than necessary. R_SNS and V_ref can be changed\n	if only significantly lower current is used\n- Vref set at constant 0.19 volts since no microstepping takes place\n- Motor current is set by PWM through V_REF pin. 100% Duty cycle \n	represents I_max motor can handle (0.6A)\n- MCU_STBY is the stepper sleep toggle used to reduce power when motors stationary"
+  (text "SCHEMATIC NOTES\n- Designed for use with Pololu SY20STH30-0604A\n- Chosen to use EN pullup instead of MCU enable control\n- MODE1 and MODE2 grounded since only full stepping is used\n- Vref/RSNS chosen for max current of 0.6A/phase, though this is\n	likely more current than necessary. R_SNS and V_ref can be changed\n	if only significantly lower current is used\n- Vref set at constant 0.19 volts since no microstepping takes place\n- Motor current is set by PWM through V_REF pin. 100% Duty cycle \n	represents I_max motor can handle (0.6A)\n- MCU_STBY is the stepper sleep toggle used to reduce power when motors stationary"
     (at 20.574 191.008 0)
     (effects (font (size 1.27 1.27)) (justify left bottom))
