File: Electrical/SADA_Board/SADA_Board/SADA_Board.kicad_sch (KiCad schematic)
At the start: 39 parts, among them J1 Headers, J2 Aux. Photodiode Board 1, J3 Aux. Photodiode Board 2, J4 Conn_01x05, J5 Systems Board Connector, U1 STM32L476RGTx, Y1 ECS_Chrystal_

Commit message: layout prog
Parts:
- removed D4, D5: TVS, Diode_SMD:D_0402_1005Metric, symbol Diode:ESD5Zxx
- J4: footprint Connector_PinSocket_2.00mm:PinSocket_1x05_P2.00mm_Vertical -> Connector_PinHeader_2.00mm:PinHeader_1x05_P2.00mm_Vertical_SMD_Pin1Left; MPN M22-2510505 -> 2PH1-10-UA-SMT-A
- JP1: footprint Connector_PinHeader_2.54mm:PinHeader_1x03_P2.54mm_Vertical_SMD_Pin1Right -> Connector_PinHeader_2.00mm:PinHeader_1x03_P2.00mm_Vertical_SMD_Pin1Left; MPN 10129380-908001BLF -> 2PH1-10-UA-SMT-A
Connections:
- net PA4 renamed DAC_OUT1
- net PA5 renamed DAC_OUT2

Commit message: layout prog
Parts:
- added R32: 270, Resistor_SMD:R_0402_1005Metric, symbol Device:R_US
- C1: value 10uF Tan. -> 10uF
- C4: value 1uF Tan. -> 1uF
- D28: value LG_R971-KN-1 -> LTST-C193KRKT-5A; footprint digikey-footprints:0805 -> LED_SMD:LED_0603_1608Metric; Category Optoelectronics -> (none); DK_Datasheet_Link https://dammedia.osram.info/media/resource/hires/osram-dam-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 -> (none); DK_Detail_Page /product-detail/en/osram-opto-semiconductors-inc/LG-R971-KN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 -> (none); Digi-Key_PN 475-1410-1-ND -> (none); Family LED Indication - Discrete -> (none); MPN LG R971-KN-1 -> LTST-C193KRKT-5A; Manufacturer OSRAM Opto Semiconductors Inc. -> (none); Status Active -> (none)
Connections:
- net GND: now also R32.2; no longer D28.2
- new net: D28.2, R32.1
Other:
- note added: "SCHEMATIC NOTES - See subpages for specific notes - BATT+ ranges 3.6V to 4.2V depending on SOC - Passive Retainment: 3" Nichrome Wire used is about 1 ohm - 'Headers' section will not be included on a final board, just for troubleshooting - Do not solder I2C pullups if included on the systems board that SADA Board interfaces with"
- note removed: "SCHEMATIC NOTES - See subpages for specific notes - BATT+ ranges 3.6V to 4.2V depending on SOC - Passive Retainment: 3" Nichrome Wire used is about 1 ohm - 'Headers' section will not be included on a final board, just for troubleshooting"
- moved on the sheet: D28

Commit message: Layout rough draft
Parts:
- removed J1: Headers, Connector_PinSocket_2.00mm:PinSocket_2x30_P2.00mm_Vertical, symbol Connector_Generic:Conn_02x30_Counter_Clockwise
- removed J2: Aux. Photodiode Board 1, Miles Added:1719730004, symbol Connector_Generic:Conn_01x04
- removed J3: Aux. Photodiode Board 2, Miles Added:1719730004, symbol Connector_Generic:Conn_01x04
- removed J5: Systems Board Connector, Miles Added:1719730004, symbol Connector_Generic:Conn_01x04
- removed TP3, TP4: TestPoint, TestPoint:TestPoint_Pad_D1.0mm, symbol Connector:TestPoint
- added J1: Conn_02x08_Odd_Even, Connector_PinHeader_2.00mm:PinHeader_2x08_P2.00mm_Vertical, symbol Connector_Generic:Conn_02x08_Odd_Even
- added J14, J15: Conn_01x02, Connector_PinSocket_2.00mm:PinSocket_1x02_P2.00mm_Vertical, symbol Connector_Generic:Conn_01x02
- added J2, J3, J5: 70543-0108, SHDR4W64P0X254_1X4_1271X508X1181P, symbol 70543-0108:70543-0108
- added S1: KSR253GLFG, KSR253GLFG, symbol KSR253GLFG:KSR253GLFG
- JP1: footprint Connector_PinHeader_2.00mm:PinHeader_1x03_P2.00mm_Vertical_SMD_Pin1Left -> Connector_PinHeader_2.00mm:PinHeader_1x03_P2.00mm_Vertical
Connections:
- net PD2 is gone; now on net Burn_sig: U1.54 (PD2)
- net +3V3: now also J1.1 (Pin_1)
- net BATT +: now also J1.15 (Pin_15), J2.3, J3.3
- net BOOT: now also J5.3
- net Burn_sig: now also J1.12 (Pin_12); no longer U1.11 (PC3)
- net DAC_OUT1: now also J15.2 (Pin_2)
- net DAC_OUT2: now also J15.1 (Pin_1)
- net GND: now also J1.16 (Pin_16), J2.4, J3.4, S1.2 (NO)
- net NRST: now also J5.4, S1.1 (COM)
- net PA6: now also J1.4 (Pin_4)
- net PA7: now also J1.2 (Pin_2)
- net PB10: now also J14.1 (Pin_1)
- net PB11: now also J14.2 (Pin_2)
- net PC13 (RTC): now also J1.7 (Pin_7)
- net PC14 (RTC): now also J1.5 (Pin_5)
- net PC15 (RTC): now also J1.3 (Pin_3)
- net PR_EN: now also J1.14 (Pin_14)
- net SYS_SCL: now also J1.11 (Pin_11), J2.1, J3.1, J5.1
- net SYS_SDA: now also J1.13 (Pin_13), J2.2, J3.2, J5.2
- net PA0: no longer names the net of U1.14 (PA0)
- net PA1: no longer names the net of U1.15 (PA1)
- net PA10: no longer names the net of U1.43 (PA10)
- net PA2: no longer names the net of U1.16 (PA2)
- net PA3: no longer names the net of U1.17 (PA3)
- net PA8: no longer names the net of U1.41 (PA8)
- net PA9: no longer names the net of U1.42 (PA9)
- net PB12: no longer names the net of U1.33 (PB12)
- net PB13: no longer names the net of U1.34 (PB13)
- net PB14: no longer names the net of U1.35 (PB14)
- net PC10: no longer names the net of U1.51 (PC10)
- net PC11: no longer names the net of U1.52 (PC11)
- net PC12: no longer names the net of U1.53 (PC12)
- net PC4: no longer names the net of U1.24 (PC4)
- net USB_OTG_FS_DM renamed USB_OTG_FS_DN
- no-connect marks 0 -> 19
Other:
- sheet USB and MCU LDO ports: added USB_OTG_FS_DN; removed USB_OTG_FS_DM
- note added: "Mounting Holes"
- note added: "Reset Switch"
- note added: "TVS diodes? pins only used on earth charge could still build up though right?"
- note removed: "TVS Diodes on clock?"
- note removed: "TVS diodes? pins only used on ground charge could still build up though right?"
- moved on the sheet: C1, C2, C3, C4, C5, C6, C7, C8, C9, D1, D2, D28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

Commit message: V1.0 Finished
Submitted to manufacturing.
Other:
- moved on the sheet: EXT3
Changed lines of the file:
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@@
     (stroke (width 0) (type default) (color 0 0 0 0))
   )
-  (polyline (pts (xy 224.028 113.919) (xy 263.398 113.919))
+  (polyline (pts (xy 223.774 118.618) (xy 265.43 118.618))
     (stroke (width 0) (type default) (color 0 0 0 0))
   )
@@
     (stroke (width 0) (type default) (color 0 0 0 0))
   )
-  (polyline (pts (xy 224.282 64.008) (xy 224.028 113.919))
+  (polyline (pts (xy 224.282 64.008) (xy 223.774 118.618))
     (stroke (width 0) (type default) (color 0 0 0 0))
   )
@@
     (stroke (width 0) (type default) (color 0 0 0 0))
   )
-  (polyline (pts (xy 263.398 113.919) (xy 263.652 64.008))
+  (polyline (pts (xy 265.43 118.618) (xy 265.176 64.008))
     (stroke (width 0) (type default) (color 0 0 0 0))
   )
@@
     (stroke (width 0) (type default) (color 0 0 0 0))
   )
-  (polyline (pts (xy 224.282 64.008) (xy 263.652 64.008))
+  (polyline (pts (xy 224.282 64.008) (xy 265.176 64.008))
     (stroke (width 0) (type default) (color 0 0 0 0))
   )
@@
     (pin "1")
   )
-  (symbol (lib_id "0_custom:{lt}name{gt}") (at 267.716 107.696 270) (unit 1)
+  (symbol (lib_id "0_custom:{lt}name{gt}") (at 269.748 107.188 270) (unit 1)
     (in_bom yes) (on_board yes)
-    (property "Reference" "EXT3" (id 0) (at 270.256 106.4259 90)
+    (property "Reference" "EXT3" (id 0) (at 272.288 105.9179 90)
       (effects (font (size 1.27 1.27)) (justify left))
     )
-    (property "Value" "Male Conn." (id 1) (at 270.256 108.9659 90)
+    (property "Value" "Male Conn." (id 1) (at 272.288 108.4579 90)
       (effects (font (size 1.27 1.27)) (justify left))
     )
-    (property "Footprint" "0_custom:EXT_no_footprint" (id 2) (at 267.716 107.696 0)
-      (effects (font (size 1.27 1.27)) hide)
-    )
-    (property "Datasheet" "" (id 3) (at 267.716 107.696 0)
-      (effects (font (size 1.27 1.27)) hide)
-    )
-    (property "MPN" "0014562042" (id 4) (at 267.716 107.696 0)
-      (effects (font (size 1.27 1.27)) hide)
-    )
+    (property "Footprint" "0_custom:EXT_no_footprint" (id 2) (at 269.748 107.188 0)
+      (effects (font (size 1.27 1.27)) hide)
+    )
+    (property "Datasheet" "" (id 3) (at 269.748 107.188 0)
+      (effects (font (size 1.27 1.27)) hide)
+    )
+    (property "MPN" "0014562042" (id 4) (at 269.748 107.188 0)
+      (effects (font (size 1.27 1.27)) hide)
+    )

Commit message: Updated BOM
Parts:
- C2: value CL1 -> 4pF
- C7: value 10 nF -> 10nF
- C9: value CL2 -> 4pF
- J2, J3, J5: MPN (none) -> 70543-0108; Manufacturer_Part_Number 70543-0108 -> (none)

Commit message: Upd. Schem and Datasheets
Parts:
- U1: value STM32L476RGTx -> STM32L476RGT3
- Y1: value ECS_Chrystal_ -> ECS-160-8-36Q-AES-TR
Changed lines of the file:
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@@
   )
   (symbol (lib_id "70543-0108:70543-0108") (at 199.136 138.938 0) (unit 1)
-    (in_bom yes) (on_board yes) (fields_autoplaced)
+    (in_bom yes) (on_board yes)
     (property "Reference" "J2" (id 0) (at 215.392 141.4779 0)
       (effects (font (size 1.27 1.27)) (justify left))
     )
-    (property "Value" "70543-0108" (id 1) (at 215.392 144.0179 0)
-      (effects (font (size 1.27 1.27)) (justify left) hide)
+    (property "Value" "70543-0108" (id 1) (at 203.454 150.622 0)
+      (effects (font (size 1.27 1.27)) (justify left))
     )
     (property "Footprint" "SHDR4W64P0X254_1X4_1271X508X1181P" (id 2) (at 215.646 136.398 0)
@@
   )
   (symbol (lib_id "70543-0108:70543-0108") (at 233.172 139.192 0) (unit 1)
-    (in_bom yes) (on_board yes) (fields_autoplaced)
+    (in_bom yes) (on_board yes)
     (property "Reference" "J3" (id 0) (at 249.428 141.7319 0)
       (effects (font (size 1.27 1.27)) (justify left))
     )
-    (property "Value" "70543-0108" (id 1) (at 249.428 144.2719 0)
-      (effects (font (size 1.27 1.27)) (justify left) hide)
+    (property "Value" "70543-0108" (id 1) (at 237.236 150.876 0)
+      (effects (font (size 1.27 1.27)) (justify left))
     )
     (property "Footprint" "SHDR4W64P0X254_1X4_1271X508X1181P" (id 2) (at 249.682 136.652 0)
@@
       (effects (font (size 1.27 1.27)) (justify left))
     )
-    (property "Value" "STM32L476RGTx" (id 1) (at 71.3614 149.86 0)
+    (property "Value" "STM32L476RGT3" (id 1) (at 71.3614 149.86 0)
       (effects (font (size 1.27 1.27)) (justify left))
     )
@@
   )
   (symbol (lib_id "70543-0108:70543-0108") (at 245.364 103.886 0) (unit 1)
-    (in_bom yes) (on_board yes) (fields_autoplaced)
+    (in_bom yes) (on_board yes)
     (property "Reference" "J5" (id 0) (at 261.62 106.4259 0)
       (effects (font (size 1.27 1.27)) (justify left))
     )
-    (property "Value" "70543-0108" (id 1) (at 261.62 108.9659 0)
-      (effects (font (size 1.27 1.27)) (justify left) hide)
+    (property "Value" "70543-0108" (id 1) (at 249.682 115.824 0)
+      (effects (font (size 1.27 1.27)) (justify left))
     )
     (property "Footprint" "SHDR4W64P0X254_1X4_1271X508X1181P" (id 2) (at 261.874 101.346 0)
@@
       (effects (font (size 1.27 1.27)) (justify left))
     )
-    (property "Value" "ECS_Chrystal_" (id 1) (at 132.334 42.164 0)
-      (effects (font (size 1.27 1.27)) hide)
-    )
+    (property "Value" "ECS-160-8-36Q-AES-TR" (id 1) (at 132.334 42.164 0))
     (property "Footprint" "Miles Added:XTAL_ECS-160-8-36Q-AES-TR" (id 2) (at 148.844 42.164 0)
       (effects (font (size 1.27 1.27)) hide)
@@
     )
     (path "/78cc26c5-c3b4-4327-b4da-d942c5c7ab26"
-      (reference "U1") (unit 1) (value "STM32L476RGTx") (footprint "Package_QFP:LQFP-64_10x10mm_P0.5mm")
+      (reference "U1") (unit 1) (value "STM32L476RGT3") (footprint "Package_QFP:LQFP-64_10x10mm_P0.5mm")
     )
     (path "/7aa0e0d2-8277-49d9-8446-a7cf9d365f33/afa449ac-389d-4002-af92-e6b269d67458"
@@
     )
     (path "/fbe0b525-e576-4e2f-9a21-465d8e24f8de"
-      (reference "Y1") (unit 1) (value "ECS_Chrystal_") (footprint "Miles Added:XTAL_ECS-160-8-36Q-AES-TR")
-    )
-  )
+      (reference "Y1") (unit 1) (value "ECS-160-8-36Q-AES-TR") (footprint "Miles Added:XTAL_ECS-160-8-36Q-AES-TR")
+    )
+  )
