File: Electrical/SADA_Board/SADA_Board/usb_MCU_LDO.kicad_sch (KiCad schematic)
At the start: 38 parts, among them IC1 TPS25940LRVCR, IC2 LP5912Q3.3DRVRQ1, J7 105431-1202, J8 10103594-0001LF, Q1 NVR5198NLT1G, Q2 NVR5198NLT1G, U11 USBLC6-2SC6, U4 NCV68261MTWAITBG, U5 NCV68261MTWAITBG

Commit message: Layout rough draft
Connections:
- net USB_CONN_DM renamed USB_CONN_DN
- net USB_OTG_FS_DM renamed USB_OTG_FS_DN
Changed lines of the file:
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@@
     (effects (font (size 1.27 1.27)) (justify right bottom))
   )
-  (label "USB_CONN_DM" (at 145.542 42.926 0)
+  (label "USB_CONN_DN" (at 145.542 42.926 0)
     (effects (font (size 1.27 1.27)) (justify left bottom))
   )
@@
     (effects (font (size 1.27 1.27)) (justify right bottom))
   )
-  (label "USB_CONN_DM" (at 139.7 34.544 180)
+  (label "USB_CONN_DN" (at 139.7 34.544 180)
     (effects (font (size 1.27 1.27)) (justify right bottom))
   )
@@
     (effects (font (size 1.27 1.27)) (justify left))
   )
-  (hierarchical_label "USB_OTG_FS_DM" (shape input) (at 160.528 37.846 180)
+  (hierarchical_label "USB_OTG_FS_DN" (shape input) (at 160.528 37.846 180)
     (effects (font (size 1.27 1.27)) (justify right))
   )

Commit message: Updated BOM
Parts:
- C14: value C -> 1.5nF
- C17, C18: value 1 uF -> 1uF
- IC2: MPN (none) -> LP5912Q3.3DRVRQ1; Manufacturer_Part_Number LP5912Q3.3DRVRQ1 -> (none)
- J7: MPN (none) -> 105431-1202; Manufacturer_Part_Number 105431-1202 -> (none)
- U11: MPN (none) -> USBLC6-2SC6
Other:
- company: (none) -> Cal Poly, SLO
- title: (none) -> CubeSat SADA - Main
Changed lines of the file:
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@@
 (kicad_sch (version 20211123) (generator eeschema)
   (paper "A4")
+  (title_block
+    (title "CubeSat SADA - Main")
+    (date "2023-04-07")
+    (rev "V1.0")
+    (company "Cal Poly, SLO")
+  )
   (junction (at 229.616 130.048) (diameter 0) (color 0 0 0 0)
   )
@@
       (effects (font (size 1.27 1.27)) (justify left))
     )
-    (property "Value" "C" (id 1) (at 83.82 71.374 0)
+    (property "Value" "1.5nF" (id 1) (at 83.82 71.374 0)
       (effects (font (size 1.27 1.27)) (justify left))
     )
@@
   (symbol (lib_id "Device:C") (at 182.118 135.128 180) (unit 1)
     (in_bom yes) (on_board yes)
-    (property "Reference" "C17" (id 0) (at 184.023 137.668 90))
-    (property "Value" "1 uF" (id 1) (at 186.563 136.398 90))
+    (property "Reference" "C17" (id 0) (at 186.944 136.398 0))
+    (property "Value" "1uF" (id 1) (at 186.944 134.366 0))
     (property "Footprint" "Capacitor_SMD:C_0603_1608Metric" (id 2) (at 181.1528 131.318 0)
       (effects (font (size 1.27 1.27)) hide)
@@
     (in_bom yes) (on_board yes)
     (property "Reference" "C18" (id 0) (at 234.442 138.176 0))
-    (property "Value" "1 uF" (id 1) (at 239.522 138.43 0))
+    (property "Value" "1uF" (id 1) (at 239.522 138.43 0))
     (property "Footprint" "Capacitor_SMD:C_0603_1608Metric" (id 2) (at 235.7628 131.318 0)
       (effects (font (size 1.27 1.27)) hide)
@@
       (effects (font (size 1.27 1.27)) (justify left) hide)
     )
-    (property "Manufacturer_Part_Number" "105431-1202" (id 9) (at 84.582 52.324 0)
+    (property "MPN" "105431-1202" (id 9) (at 84.582 52.324 0)
       (effects (font (size 1.27 1.27)) (justify left) hide)
     )
@@
     )
     (property "Datasheet" "https://www.st.com/resource/en/datasheet/usblc6-2.pdf" (id 3) (at 175.768 31.496 0)
+      (effects (font (size 1.27 1.27)) hide)
+    )
+    (property "MPN" "USBLC6-2SC6" (id 4) (at 170.688 40.386 0)
       (effects (font (size 1.27 1.27)) hide)
     )
@@
       (effects (font (size 1.27 1.27)) (justify left) hide)
     )
-    (property "Manufacturer_Part_Number" "LP5912Q3.3DRVRQ1" (id 9) (at 202.946 145.288 0)
-      (effects (font (size 1.27 1.27)) (justify left) hide)
-    )
+    (property "MPN" "LP5912Q3.3DRVRQ1" (id 9) (at 202.946 145.288 0)
+      (effects (font (size 1.27 1.27)) (justify left) hide)
+    )

Commit message: Upd. Schem and Datasheets
Changed lines of the file:
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@@
   )
   (symbol (lib_name "NCV68261MTWAITBG_1") (lib_id "Ideal_diode_NCV:NCV68261MTWAITBG") (at 214.376 87.63 0) (unit 1)
-    (in_bom yes) (on_board yes) (fields_autoplaced)
+    (in_bom yes) (on_board yes)
     (property "Reference" "U5" (id 0) (at 214.376 77.47 0)
       (effects (font (size 1.524 1.524)))
     )
-    (property "Value" "NCV68261MTWAITBG" (id 1) (at 214.376 81.28 0)
+    (property "Value" "NCV68261MTWAITBG" (id 1) (at 214.376 80.518 0)
       (effects (font (size 1.524 1.524)))
     )
