File: Electrical/Photodiode Breakout/Photodiode_Board/Photodiode_Board.kicad_sch (KiCad schematic)
At the start: 12 parts, among them U1 CD4051B, U2 LM358

Commit message: Layout rough draft
Parts:
- removed D1, D2, D3, D4: BPW34, OptoDevice:Osram_BPW34S-SMD, symbol Sensor_Optical:BPW34-SMD
- removed R1, R2, R3, R4: 1M, symbol Device:R_US
- removed R5: 10k, symbol Device:R_US
- removed R6: 180k, symbol Device:R_US
- removed U1: CD4051B, symbol Analog_Switch:CD4051B
- removed U2: LM358, symbol Amplifier_Operational:LM358
- added C?: 10 nF, Capacitor_SMD:C_0402_1005Metric, symbol Device:C
- added C?: 1nF, Resistor_SMD:R_0402_1005Metric, symbol Device:C
- added D?: TVS, Diode_SMD:D_0402_1005Metric, symbol Diode:ESD5Zxx
- added EXT?: Male Conn., 0_custom:EXT_no_footprint, symbol 0_custom:{lt}name{gt}
- added IC?: TPS79333DBVRQ1, SOT95P280X145-5N, symbol TPS79333DBVRQ1:TPS79333DBVRQ1
- added J?: 70543-0108, SHDR4W64P0X254_1X4_1271X508X1181P, symbol 70543-0108:70543-0108
- added R?: 200k, Resistor_SMD:R_0603_1608Metric_Pad0.98x0.95mm_HandSolder, symbol Device:R_US
- added TP? (x2): TestPoint, TestPoint:TestPoint_Pad_D1.0mm, symbol Connector:TestPoint
- added U?: LM321, Package_TO_SOT_SMD:SOT-23-5, symbol Amplifier_Operational:LMV321
- added U?: CD4051B, Miles Added:PW0016A_L, symbol Analog_Switch:CD4051B
Connections:
- net GND: now also C?.2, D?.2 (A), J?.4, U?.1 (+), U?.2 (V-), U?.6 (INH), U?.7 (VEE), U?.8 (VSS)
- net MCU ADC: now also U?.4
- new net: C?.1, C?.2, D?.1 (K), R?.1, TP?.1, U?.3 (-), U?.3 (X)
- new net: C?.1, R?.2, TP?.1
- new net +3V3: U?.16 (VDD), U?.5 (V+)
- new net BATT +: J?.3
- new net MUX (S0): U?.11 (A)
- new net MUX (S1): U?.10 (B)
- new net MUX (S2): U?.9 (C)
- new net PhDio_0: U?.13 (X0)
- new net PhDio_1: U?.14 (X1)
- new net PhDio_2: U?.15 (X2)
- new net PhDio_3: U?.12 (X3)
- new net PhDio_4: U?.1 (X4)
- new net PhDio_5: U?.5 (X5)
- new net PhDio_6: U?.2 (X6)
- new net PhDio_7: U?.4 (X7)
- new net SYS_SCL: J?.1
- new net SYS_SDA: J?.2

Commit message: Upd. Schem and Datasheets
Parts:
- added D?: D_Photo, Diode_SMD:D_0805_2012Metric, symbol Device:D_Photo
Changed lines of the file:
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@@
     (pin "1")
+  )
+  (symbol (lib_id "Device:D_Photo") (at 218.44 96.266 0) (unit 1)
+    (in_bom yes) (on_board yes) (fields_autoplaced)
+    (property "Reference" "D?" (id 0) (at 217.4875 87.63 0))
+    (property "Value" "D_Photo" (id 1) (at 217.4875 90.17 0))
+    (property "Footprint" "Diode_SMD:D_0805_2012Metric" (id 2) (at 217.17 96.266 0)
+      (effects (font (size 1.27 1.27)) hide)
+    )
+    (property "Datasheet" "~" (id 3) (at 217.17 96.266 0)
+      (effects (font (size 1.27 1.27)) hide)
+    )
+    (property "MPN" "VEMD1060X01" (id 4) (at 218.44 96.266 0)
+      (effects (font (size 1.27 1.27)) hide)
+    )
+    (pin "1")
+    (pin "2")
   )
   (symbol (lib_id "power:+3V3") (at 118.872 120.142 90) (unit 1)
@@
       (reference "C?") (unit 1) (value "1nF") (footprint "Resistor_SMD:R_0402_1005Metric")
     )
+    (path "/e5b7ae6f-7c5f-445f-9053-e1513fadff38"
+      (reference "D?") (unit 1) (value "D_Photo") (footprint "Diode_SMD:D_0805_2012Metric")
+    )
     (path "/f99ae1b0-bde7-4db2-b184-e4935509a461"

Commit message: PhDio Rough Schem
Parts:
- removed C?: 10 nF, Capacitor_SMD:C_0402_1005Metric, symbol Device:C
- removed C?: 1nF, Resistor_SMD:R_0402_1005Metric, symbol Device:C
- removed D?: D_Photo, Diode_SMD:D_0805_2012Metric, symbol Device:D_Photo
- removed IC?: TPS79333DBVRQ1, SOT95P280X145-5N, symbol TPS79333DBVRQ1:TPS79333DBVRQ1
- removed R?: 200k, Resistor_SMD:R_0603_1608Metric_Pad0.98x0.95mm_HandSolder, symbol Device:R_US
- removed TP? (x2): TestPoint, TestPoint:TestPoint_Pad_D1.0mm, symbol Connector:TestPoint
- removed U?: LM321, Package_TO_SOT_SMD:SOT-23-5, symbol Amplifier_Operational:LMV321
- removed U?: CD4051B, Miles Added:PW0016A_L, symbol Analog_Switch:CD4051B
- added C1, C3: 2.2 uF, Resistor_SMD:R_0603_1608Metric, symbol Device:C
- added C2: 1uF, Capacitor_SMD:C_0603_1608Metric, symbol Device:C
- added C4: 10uF, Capacitor_SMD:C_0603_1608Metric, symbol Device:C
- added C5, C6: 100nF, Capacitor_SMD:C_0402_1005Metric, symbol Device:C
- added D2, D3, D4, D5, D7, D8: TVS, Diode_SMD:D_0402_1005Metric, symbol Diode:ESD5Zxx
- added D6: LTST-C193KRKT-5A, LED_SMD:LED_0603_1608Metric, symbol dk_LED-Indication-Discrete:LG_R971-KN-1
- added EXT2: Male Conn., 0_custom:EXT_no_footprint, symbol 0_custom:{lt}name{gt}
- added H1, H2, H3, H4: MountingHole_Pad, MountingHole:MountingHole_2.2mm_M2_Pad_Via, symbol Mechanical:MountingHole_Pad
- added J2: 70543-0108, SHDR4W64P0X254_1X4_1271X508X1181P, symbol 70543-0108:70543-0108
- added R1, R2: 330, Resistor_SMD:R_0402_1005Metric, symbol Device:R_US
- added TP1, TP2, TP3, TP4: TestPoint, TestPoint:TestPoint_Pad_D1.0mm, symbol Connector:TestPoint
- added U1: LM2775QDSGRQ1, DSG0008A, symbol LM2775q1:LM2775QDSGRQ1
- added U2: TSL1401, Package_DIP:DIP-8_W10.16mm, symbol 0_custom:TSL1401
- added U3: MCP3221A0T-E/OT, SOT-23-5_MC_MCH, symbol MCP3221:MCP3221A0T-E/OT
- gave numbers to parts that had none: 3
Connections:
- net BATT +: now also D1.1 (K), C1.1, U1.1 (PFM), U1.4 (OUTDIS), U1.5 (EN), U1.7 (VIN)
- net GND: now also C1.2, C3.2, C4.1, C5.1, C6.1, D2.2 (A), D3.2 (A), D4.2 (A), D5.2 (A), D7.2 (A), D8.2 (A), H1.1, H2.1, H3.1, H4.1, R1.2, R2.2, U1.8 (GND), U1.9 (GND), U2.6 (GND), U2.7 (GND), U3.2 (VSS)
- net SYS_SCL: now also U3.5 (SCL)
- net SYS_SDA: now also U3.4 (SDA)
- new net: C2.1, U1.2 (C1-)
- new net: C2.2, U1.3 (C1+)
- new net: D6.2, R1.1
- new net +5V: C3.1, C4.2, C5.2, C6.2, D2.1 (K), D3.1 (K), D6.1, D8.1 (K), TP1.1, U1.6 (VOUT), U2.4 (VDD), U3.1 (VDD)
- new net AO: D7.1 (K), R2.1, TP4.1, U2.3 (AO), U3.3 (A_IN)
- new net CLK: D5.1 (K), J2.2, TP3.1, U2.2 (CLK)
- new net SI: D4.1 (K), J2.1, TP2.1, U2.1 (SI)
- no-connect marks 0 -> 2
Other:
- note added: "5V Boost"
- note added: "ADC"
- note added: "Other"
- note added: "Photodiode Array"
- note added: "SADA Board Conn."
- company: (none) -> Cal Poly - SLO
- title: (none) -> CubeSat SADA - Photodiode Board
- moved on the sheet: D1, EXT1, J1
